File: Atomic_V1.0/Atomic_V1.0.sch (EAGLE design)
At the start: 14 parts, among them U4 TLE9250VSJ, X1 S4P-VH

Commit message: done Linear Regulator Version.
Parts:
- removed D2: SS12L R3, fliegl-elektronik:S1ML
- removed U1: (no value), Wurth_Step Down Converter_MagI³C-FDSM:MAGI³C-FDSM_SIP-3_173010542_173XXXX42
- added C2: 100 nF, fliegl-wuerth:WCAP-CSGP_0402_885012205037_16V(DC)
- added C3: 22 µF, Wurth_Capacitors_WCAP-CSGP:WCAP-CSGP_0805_H1.25_885012107011_10V(DC)
- added G1: TLE4270-2D-INF-PG-TO252-5-11_L_1, INF-PG-TO252-5-11L:TLE4270-2D-INF-PG-TO252-5-11_L_1
Connections:
- net +12V: now also C1.2, G1.I; no longer D2.A
- net +5V: now also C3.2, G1.Q; no longer U1.VOUT
- net GND: now also C2.2, C3.1, G1.GND; no longer U1.GND
- net N$1: now also C2.1, G1.D; no longer C1.2, D2.C, U1.VIN
Other:
- moved on the sheet: C1
Changed lines of the file:
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@@
 <layer number="91" name="Nets" color="2" fill="1" visible="yes" active="yes"/>
 <layer number="92" name="Busses" color="1" fill="1" visible="yes" active="yes"/>
-<layer number="93" name="Pins" color="2" fill="1" visible="no" active="yes"/>
+<layer number="93" name="Pins" color="2" fill="1" visible="yes" active="yes"/>
 <layer number="94" name="Symbols" color="4" fill="1" visible="yes" active="yes"/>
 <layer number="95" name="Names" color="7" fill="1" visible="yes" active="yes"/>
@@
 <part name="C17" library="fliegl-wuerth" deviceset="WCAP-CSGP_0402" device="_16V(DC)" technology="_885012205037" value="100 nF"/>
 <part name="C19" library="fliegl-wuerth" deviceset="WCAP-CSGP_0402" device="_16V(DC)" technology="_885012205037" value="100 nF"/>
-<part name="U1" library="Wurth_Step Down Converter_MagI³C-FDSM" library_urn="urn:adsk.eagle:library:13379781" deviceset="MAGI³C-FDSM_SIP-3" device="_173XXXX42" package3d_urn="urn:adsk.eagle:package:13379788/2" technology="_173010542"/>
 <part name="GND1" library="supply1" deviceset="GND" device=""/>
 <part name="GND2" library="supply1" deviceset="GND" device=""/>
@@
 <part name="P+3" library="supply1" deviceset="+5V" device=""/>
 <part name="D1" library="Wurth_EMC Components_WE-TVSP" library_urn="urn:adsk.eagle:library:14283044" deviceset="WE-TVSP_DO-214AC_400W_BI" device="" package3d_urn="urn:adsk.eagle:package:12146531/2" technology="_824501261" value="26V"/>
-<part name="D2" library="fliegl-elektronik" deviceset="S1ML" device="" value="SS12L R3"/>
 <part name="GND4" library="supply1" deviceset="GND" device=""/>
 <part name="C1" library="Wurth_Capacitors_WCAP-CSGP" library_urn="urn:adsk.eagle:library:18488985" deviceset="WCAP-CSGP_1210_H2.5" device="_25V(DC)" package3d_urn="urn:adsk.eagle:package:18489097/2" technology="_885012109014" value="47uF"/>
 <part name="GND6" library="supply1" deviceset="GND" device=""/>
+<part name="G1" library="INF-PG-TO252-5-11L" deviceset="TLE4270-2D-INF-PG-TO252-5-11_L_1" device=""/>
+<part name="C2" library="fliegl-wuerth" deviceset="WCAP-CSGP_0402" device="_16V(DC)" technology="_885012205037" value="100 nF"/>
+<part name="GND7" library="supply1" deviceset="GND" device=""/>
+<part name="C3" library="Wurth_Capacitors_WCAP-CSGP" library_urn="urn:adsk.eagle:library:18488985" deviceset="WCAP-CSGP_0805_H1.25" device="_10V(DC)" package3d_urn="urn:adsk.eagle:package:18489127/2" technology="_885012107011" value="22  µF "/>
+<part name="GND8" library="supply1" deviceset="GND" device=""/>
 </parts>
 <sheets>
@@
 <attribute name="NAME" x="-36.322" y="138.43" size="1.778" layer="95" rot="MR270"/>
 </instance>
-<instance part="U1" gate="G$1" x="38.1" y="124.46" smashed="yes">
-<attribute name="NAME" x="38.1" y="131.28" size="1.778" layer="95" align="bottom-center"/>
-<attribute name="VALUE" x="42.85" y="115.8" size="1.778" layer="96"/>
-</instance>
-<instance part="GND1" gate="1" x="38.1" y="111.76" smashed="yes" rot="MR0">
-<attribute name="VALUE" x="40.64" y="109.22" size="1.778" layer="96" rot="MR0"/>
+<instance part="GND1" gate="1" x="35.56" y="93.98" smashed="yes" rot="MR0">
+<attribute name="VALUE" x="38.1" y="91.44" size="1.778" layer="96" rot="MR0"/>
 </instance>
 <instance part="GND2" gate="1" x="-25.4" y="119.38" smashed="yes">
 <attribute name="VALUE" x="-27.94" y="114.3" size="1.778" layer="96"/>
 </instance>
-<instance part="P+3" gate="1" x="53.34" y="139.7" smashed="yes" rot="MR0">
-<attribute name="VALUE" x="55.88" y="134.62" size="1.778" layer="96" rot="MR90"/>
+<instance part="P+3" gate="1" x="48.26" y="142.24" smashed="yes" rot="MR0">
+<attribute name="VALUE" x="50.8" y="137.16" size="1.778" layer="96" rot="MR90"/>
 </instance>
 <instance part="D1" gate="G$1" x="-15.24" y="119.38" smashed="yes" rot="R90">
@@
 <attribute name="VALUE" x="-11.43" y="116.84" size="1.27" layer="95" rot="R90"/>
 </instance>
-<instance part="D2" gate="G$1" x="-7.62" y="127" smashed="yes">
-<attribute name="NAME" x="-8.89" y="129.54" size="1.778" layer="95"/>
-<attribute name="VALUE" x="-8.89" y="123.19" size="1.778" layer="96"/>
-<attribute name="ARTIKEL_NR" x="-8.89" y="120.65" size="1.27" layer="96"/>
-</instance>
 <instance part="GND4" gate="1" x="-15.24" y="111.76" smashed="yes">
 <attribute name="VALUE" x="-17.78" y="106.68" size="1.778" layer="96"/>
 </instance>
-<instance part="C1" gate="G$1" x="7.62" y="119.38" smashed="yes" rot="R90">
-<attribute name="NAME" x="4.24" y="120.555" size="1.4224" layer="95" rot="R90" align="bottom-center"/>
-<attribute name="VALUE" x="12.695" y="120.295" size="1.4224" layer="96" rot="R90" align="bottom-center"/>
-</instance>
-<instance part="GND6" gate="1" x="7.62" y="114.3" smashed="yes">
-<attribute name="VALUE" x="5.08" y="109.22" size="1.778" layer="96"/>
+<instance part="C1" gate="G$1" x="7.62" y="116.84" smashed="yes" rot="R90">
+<attribute name="NAME" x="4.24" y="118.015" size="1.4224" layer="95" rot="R90" align="bottom-center"/>
+<attribute name="VALUE" x="12.695" y="117.755" size="1.4224" layer="96" rot="R90" align="bottom-center"/>
+</instance>
+<instance part="GND6" gate="1" x="7.62" y="109.22" smashed="yes">
+<attribute name="VALUE" x="5.08" y="104.14" size="1.778" layer="96"/>
+</instance>
+<instance part="G1" gate="G" x="35.56" y="121.92" smashed="yes">
+<attribute name="NAME" x="66.04" y="117.475" size="1.778" layer="95"/>
+<attribute name="VALUE" x="66.04" y="121.92" size="1.778" layer="96"/>
+</instance>
+<instance part="C2" gate="G$1" x="48.26" y="109.22" smashed="yes" rot="MR0">
+<attribute name="NAME" x="45.72" y="109.22" size="1.778" layer="95" rot="MR0"/>
+<attribute name="VALUE" x="45.72" y="106.68" size="1.778" layer="96" rot="MR0"/>
+</instance>
+<instance part="GND7" gate="1" x="48.26" y="93.98" smashed="yes" rot="MR0">
+<attribute name="VALUE" x="50.8" y="91.44" size="1.778" layer="96" rot="MR0"/>
+</instance>
+<instance part="C3" gate="G$1" x="60.96" y="106.68" smashed="yes" rot="R90">
+<attribute name="NAME" x="57.58" y="107.855" size="1.4224" layer="95" rot="R90" align="bottom-center"/>
+<attribute name="VALUE" x="66.035" y="107.595" size="1.4224" layer="96" rot="R90" align="bottom-center"/>
+</instance>
+<instance part="GND8" gate="1" x="60.96" y="93.98" smashed="yes" rot="MR0">
+<attribute name="VALUE" x="63.5" y="91.44" size="1.778" layer="96" rot="MR0"/>
 </instance>
 </instances>
@@
 </segment>
 <segment>
-<pinref part="U1" gate="G$1" pin="GND"/>
 <pinref part="GND1" gate="1" pin="GND"/>
+<pinref part="G1" gate="G" pin="GND"/>
+<wire x1="35.56" y1="96.52" x2="35.56" y2="109.22" width="0.1524" layer="91"/>
 </segment>
 <segment>
@@
 <pinref part="C1" gate="G$1" pin="1"/>
 <pinref part="GND6" gate="1" pin="GND"/>
+<wire x1="7.62" y1="111.76" x2="7.62" y2="114.3" width="0.1524" layer="91"/>
+</segment>
+<segment>
+<pinref part="C2" gate="G$1" pin="2"/>
+<wire x1="48.26" y1="104.14" x2="48.26" y2="96.52" width="0.1524" layer="91"/>
+<pinref part="GND7" gate="1" pin="GND"/>
+</segment>
+<segment>
+<pinref part="C3" gate="G$1" pin="1"/>
+<pinref part="GND8" gate="1" pin="GND"/>
+<wire x1="60.96" y1="96.52" x2="60.96" y2="104.14" width="0.1524" layer="91"/>
 </segment>
 </net>
 <net name="+5V" class="0">
 <segment>
-<pinref part="U1" gate="G$1" pin="VOUT"/>
 <pinref part="P+3" gate="1" pin="+5V"/>
-<wire x1="53.34" y1="137.16" x2="53.34" y2="127" width="0.1524" layer="91"/>
+<pinref part="G1" gate="G" pin="Q"/>
+<wire x1="48.26" y1="139.7" x2="48.26" y2="127" width="0.1524" layer="91"/>
+<pinref part="C3" gate="G$1" pin="2"/>
+<wire x1="48.26" y1="127" x2="60.96" y2="127" width="0.1524" layer="91"/>
+<wire x1="60.96" y1="127" x2="60.96" y2="111.76" width="0.1524" layer="91"/>
+<junction x="48.26" y="127"/>
 </segment>
 </net>
@@
 <pinref part="X1" gate="G$1" pin="2"/>
 <wire x1="-27.94" y1="129.54" x2="-27.94" y2="127" width="0.1524" layer="91"/>
-<pinref part="D2" gate="G$1" pin="A"/>
-<wire x1="-10.16" y1="127" x2="-15.24" y2="127" width="0.1524" layer="91"/>
 <pinref part="D1" gate="G$1" pin="2"/>
 <wire x1="-15.24" y1="127" x2="-27.94" y2="127" width="0.1524" layer="91"/>
 <junction x="-15.24" y="127"/>
-</segment>
-</net>
-<net name="N$1" class="0">
-<segment>
-<pinref part="U1" gate="G$1" pin="VIN"/>
-<pinref part="D2" gate="G$1" pin="C"/>
-<wire x1="-5.08" y1="127" x2="7.62" y2="127" width="0.1524" layer="91"/>
+<wire x1="-15.24" y1="127" x2="7.62" y2="127" width="0.1524" layer="91"/>
 <pinref part="C1" gate="G$1" pin="2"/>
 <wire x1="7.62" y1="127" x2="22.86" y2="127" width="0.1524" layer="91"/>
-<wire x1="7.62" y1="124.46" x2="7.62" y2="127" width="0.1524" layer="91"/>
+<wire x1="7.62" y1="121.92" x2="7.62" y2="127" width="0.1524" layer="91"/>
 <junction x="7.62" y="127"/>
-</segment>
-</net>
+<pinref part="G1" gate="G" pin="I"/>
+</segment>
+</net>
+<net name="N$1" class="0">
+<segment>
+<pinref part="G1" gate="G" pin="D"/>
+<pinref part="C2" gate="G$1" pin="1"/>
+<wire x1="48.26" y1="116.84" x2="48.26" y2="111.76" width="0.1524" layer="91"/>
+</segment>
+</net>
