File: Atomic_V1.0/Atomic_V1.0.brd (EAGLE design)
At the start: 20 x 44 mm, 14 parts, among them U4 TLE9250VSJ, X1 S4P-VH

Commit message: DCDC Version
Parts:
- removed D2: SS12L R3, fliegl-elektronik:SMA
- added D3: SS12L_R3, SS12L_R3:SODFL3618X143N
- moved C1 11.0 mm to (16.0, 25.4)
- moved D6 6.86 mm to (7.62, 20.4), turned to 90 degrees
- moved U1 5.04 mm to (8.24, 30.3), turned to 180 degrees
- moved D1 1.39 mm to (0.30, 29.1)
Connections:
- net +12V: now also D3.2; no longer D2.A
- net N$1: now also D3.1; no longer D2.C
Routing:
- net +12V: track 9.70 -> 17.3 mm
- net +5V: track 30.2 -> 35.8 mm
- net CAN_H: track 30.5 -> 28.0 mm
- net CAN_L: track 30.6 -> 28.3 mm
- net GND: vias 45 -> 49

Commit message: ..
Parts:
- moved D1 0.73 mm to (0.30, 28.3)
Changed lines of the file:
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@@
 <attribute name="VALUE" x="11.74" y="34.285" size="1.27" layer="27" rot="R180"/>
 </element>
-<element name="D1" library="Wurth_EMC Components_WE-TVSP" library_urn="urn:adsk.eagle:library:14283044" package="WE-TVSP_DO-214AC_BIDIRECTIONAL" package3d_urn="urn:adsk.eagle:package:12146531/2" value="26V" x="0.299" y="29.053" smashed="yes" rot="R90">
-<attribute name="DATASHEET-URL" value="https://katalog.we-online.com/pbs/datasheet/824501261.pdf" x="0.299" y="29.053" size="1.778" layer="27" rot="R90" display="off"/>
-<attribute name="IPEAK" value="9.5A" x="0.299" y="29.053" size="1.778" layer="27" rot="R90" display="off"/>
-<attribute name="MOUNT" value="SMT" x="0.299" y="29.053" size="1.778" layer="27" rot="R90" display="off"/>
-<attribute name="NAME" x="-1.46" y="29.688" size="0.8" layer="25" rot="R90" align="bottom-center"/>
-<attribute name="PART-NUMBER" value=" 824501261 " x="0.299" y="29.053" size="1.778" layer="27" rot="R90" display="off"/>
-<attribute name="PDISS" value="400W" x="0.299" y="29.053" size="1.778" layer="27" rot="R90" display="off"/>
-<attribute name="VALUE" x="-1.39" y="26.343" size="1.016" layer="27" rot="R90"/>
-<attribute name="VBR" value="30.4V" x="0.299" y="29.053" size="1.778" layer="27" rot="R90" display="off"/>
-<attribute name="VCLAMP" value="42.1V" x="0.299" y="29.053" size="1.778" layer="27" rot="R90" display="off"/>
+<element name="D1" library="Wurth_EMC Components_WE-TVSP" library_urn="urn:adsk.eagle:library:14283044" package="WE-TVSP_DO-214AC_BIDIRECTIONAL" package3d_urn="urn:adsk.eagle:package:12146531/2" value="26V" x="0.299" y="28.321" smashed="yes" rot="R90">
+<attribute name="DATASHEET-URL" value="https://katalog.we-online.com/pbs/datasheet/824501261.pdf" x="0.299" y="28.321" size="1.778" layer="27" rot="R90" display="off"/>
+<attribute name="IPEAK" value="9.5A" x="0.299" y="28.321" size="1.778" layer="27" rot="R90" display="off"/>
+<attribute name="MOUNT" value="SMT" x="0.299" y="28.321" size="1.778" layer="27" rot="R90" display="off"/>
+<attribute name="NAME" x="-1.46" y="28.956" size="0.8" layer="25" rot="R90" align="bottom-center"/>
+<attribute name="PART-NUMBER" value=" 824501261 " x="0.299" y="28.321" size="1.778" layer="27" rot="R90" display="off"/>
+<attribute name="PDISS" value="400W" x="0.299" y="28.321" size="1.778" layer="27" rot="R90" display="off"/>
+<attribute name="VALUE" x="-1.39" y="25.611" size="1.016" layer="27" rot="R90"/>
+<attribute name="VBR" value="30.4V" x="0.299" y="28.321" size="1.778" layer="27" rot="R90" display="off"/>
+<attribute name="VCLAMP" value="42.1V" x="0.299" y="28.321" size="1.778" layer="27" rot="R90" display="off"/>
 </element>
 <element name="C1" library="Wurth_Capacitors_WCAP-CSGP" library_urn="urn:adsk.eagle:library:18488985" package="WCAP-CSGP_1210_H2.5" package3d_urn="urn:adsk.eagle:package:18489097/2" value="47uF" x="16.042" y="25.356" smashed="yes" rot="R90">
@@
 <wire x1="9.6" y1="33.92" x2="9.966" y2="33.92" width="1.27" layer="1"/>
 <wire x1="12.197" y1="31.689" x2="15.499" y2="31.689" width="1.27" layer="1"/>
-<wire x1="0.9666" y1="31.8206" x2="0.299" y2="31.153" width="1.1" layer="1"/>
+<wire x1="1.6986" y1="31.8206" x2="0.299" y2="30.421" width="1.1" layer="1"/>
 <wire x1="9.6" y1="33.92" x2="8.975" y2="33.92" width="1.1" layer="1"/>
 <wire x1="8.975" y1="33.92" x2="6.8756" y2="31.8206" width="1.1" layer="1"/>
-<wire x1="6.8756" y1="31.8206" x2="0.9666" y2="31.8206" width="1.1" layer="1"/>
+<wire x1="6.8756" y1="31.8206" x2="1.6986" y2="31.8206" width="1.1" layer="1"/>
 </signal>
 <signal name="N$1">
