File: Atomic_V1.0/Atomic_V1.0_LDO.brd (EAGLE design)
At the start: 20 x 44 mm, 14 parts, among them U4 TLE9250VSJ, X1 S4P-VH

Commit message: merge
Parts:
- removed D3: SS12L_R3, SS12L_R3:SODFL3618X143N
- removed U1: (no value), Wurth_Step Down Converter_MagI³C-FDSM:MAGI³C-FDSM_173XXXX42
- added C2: 100 nF, fliegl-wuerth:WCAP-CSGP_0402
- added C3: 22 µF, Wurth_Capacitors_WCAP-CSGP:WCAP-CSGP_0805_H1.25_R
- added G1: TLE4270-2D-INF-PG-TO252-5-11_L_1, INF-PG-TO252-5-11L:INF-PG-TO252-5-11_L_1PRIMARY
- moved C1 9.04 mm to (7.11, 26.7), turned to 0 degrees
- moved D1 6.58 mm to (6.58, 30.3), turned to 0 degrees
- moved D6 4.46 mm to (3.56, 22.2)
Connections:
- net +12V: now also C1.2, G1.1; no longer D3.2
- net +5V: now also C3.2, G1.5; no longer U1.3
- net GND: now also C2.2, C3.1, G1.3; no longer U1.2
- net N$1: now also C2.1, G1.4; no longer C1.2, D3.1, U1.1
Routing:
- net GND: track 2.24 -> 12.2 mm, vias 49 -> 97
- net CAN_L: track 28.3 -> 33.7 mm
- net +12V: track 17.6 -> 13.8 mm
- net N$1: track 7.33 -> 5.92 mm
- net CAN_H: track 28.0 -> 29.4 mm
- net +5V: track 35.8 -> 37.0 mm, vias 1 -> 4
