File: Atomic_V1.0/Atomic_Stick.sch (EAGLE design)
At the start: 14 parts, among them U4 TLE9250VSJ

Commit message: ..
Parts:
- added J3, J4: (no value), Wurth_Connectors_WR-LECO:695402400222
Connections:
- net +12V: now also J3.2
- net CAN_H: now also J3.1
- net CAN_L: now also J4.2
- net GND: now also J4.1
Other:
- note removed: "G"
- note removed: "H"
- note removed: "L"
- note removed: "V"
Changed lines of the file:
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@@
 <part name="C3" library="Wurth_Capacitors_WCAP-CSGP" library_urn="urn:adsk.eagle:library:18488985" deviceset="WCAP-CSGP_0805_H1.25" device="_10V(DC)" package3d_urn="urn:adsk.eagle:package:18489127/2" technology="_885012107011" value="22  µF "/>
 <part name="GND8" library="supply1" deviceset="GND" device=""/>
+<part name="J3" library="Wurth_Connectors_WR-LECO" library_urn="urn:adsk.eagle:library:14873884" deviceset="695402400222" device="" package3d_urn="urn:adsk.eagle:package:14873908/2"/>
+<part name="J4" library="Wurth_Connectors_WR-LECO" library_urn="urn:adsk.eagle:library:14873884" deviceset="695402400222" device="" package3d_urn="urn:adsk.eagle:package:14873908/2"/>
 </parts>
 <sheets>
 <sheet>
 <plain>
-<text x="-25.4" y="139.7" size="1.778" layer="95">G</text>
-<text x="-27.94" y="139.7" size="1.778" layer="95">V</text>
-<text x="-30.48" y="139.7" size="1.778" layer="95">H</text>
-<text x="-33.02" y="139.7" size="1.778" layer="95">L</text>
 <frame x1="-104.14" y1="-20.32" x2="281.94" y2="198.12" columns="8" rows="5" layer="94"/>
 </plain>
@@
 <attribute name="VALUE" x="38.1" y="91.44" size="1.778" layer="96" rot="MR0"/>
 </instance>
-<instance part="GND2" gate="1" x="-25.4" y="119.38" smashed="yes">
-<attribute name="VALUE" x="-27.94" y="114.3" size="1.778" layer="96"/>
+<instance part="GND2" gate="1" x="-35.56" y="134.62" smashed="yes">
+<attribute name="VALUE" x="-38.1" y="129.54" size="1.778" layer="96"/>
 </instance>
 <instance part="P+3" gate="1" x="48.26" y="142.24" smashed="yes" rot="MR0">
@@
 <attribute name="VALUE" x="63.5" y="91.44" size="1.778" layer="96" rot="MR0"/>
 </instance>
+<instance part="J3" gate="G$1" x="-38.1" y="157.48" smashed="yes">
+<attribute name="NAME" x="-42.98" y="156.558" size="1.016" layer="95" align="bottom-right"/>
+<attribute name="VALUE" x="-42.93" y="154.9" size="1.016" layer="96" align="bottom-right"/>
+</instance>
+<instance part="J4" gate="G$1" x="-33.02" y="147.32" smashed="yes">
+<attribute name="NAME" x="-37.9" y="146.398" size="1.016" layer="95" align="bottom-right"/>
+<attribute name="VALUE" x="-37.85" y="144.74" size="1.016" layer="96" align="bottom-right"/>
+</instance>
 </instances>
 <busses>
@@
 <net name="GND" class="1">
 <segment>
-<wire x1="-25.4" y1="129.54" x2="-25.4" y2="121.92" width="0.1524" layer="91"/>
+<wire x1="-35.56" y1="142.24" x2="-35.56" y2="137.16" width="0.1524" layer="91"/>
 <label x="-27.94" y="111.76" size="1.778" layer="95"/>
 <pinref part="GND2" gate="1" pin="GND"/>
+<pinref part="J4" gate="G$1" pin="1"/>
 </segment>
 <segment>
@@
 <net name="CAN_H" class="0">
 <segment>
-<wire x1="-30.48" y1="129.54" x2="-30.48" y2="119.38" width="0.1524" layer="91"/>
-<wire x1="-30.48" y1="119.38" x2="-43.18" y2="119.38" width="0.1524" layer="91"/>
-<label x="-43.18" y="119.38" size="1.778" layer="95" rot="R180" xref="yes"/>
+<wire x1="-40.64" y1="152.4" x2="-40.64" y2="142.24" width="0.1524" layer="91"/>
+<wire x1="-40.64" y1="142.24" x2="-45.72" y2="142.24" width="0.1524" layer="91"/>
+<label x="-45.72" y="142.24" size="1.778" layer="95" rot="R180" xref="yes"/>
+<pinref part="J3" gate="G$1" pin="1"/>
 </segment>
 </net>
 <net name="CAN_L" class="0">
 <segment>
-<wire x1="-33.02" y1="129.54" x2="-33.02" y2="127" width="0.1524" layer="91"/>
+<wire x1="-33.02" y1="142.24" x2="-33.02" y2="127" width="0.1524" layer="91"/>
 <wire x1="-33.02" y1="127" x2="-43.18" y2="127" width="0.1524" layer="91"/>
 <label x="-43.18" y="127" size="1.778" layer="95" rot="R180" xref="yes"/>
+<pinref part="J4" gate="G$1" pin="2"/>
 </segment>
 </net>
 <net name="+12V" class="0">
 <segment>
-<wire x1="-27.94" y1="129.54" x2="-27.94" y2="127" width="0.1524" layer="91"/>
 <pinref part="D1" gate="G$1" pin="2"/>
-<wire x1="-15.24" y1="127" x2="-27.94" y2="127" width="0.1524" layer="91"/>
 <junction x="-15.24" y="127"/>
 <wire x1="-15.24" y1="127" x2="7.62" y2="127" width="0.1524" layer="91"/>
@@
 <junction x="7.62" y="127"/>
 <pinref part="G1" gate="G" pin="I"/>
+<pinref part="J3" gate="G$1" pin="2"/>
+<wire x1="-38.1" y1="152.4" x2="-15.24" y2="152.4" width="0.1524" layer="91"/>
+<wire x1="-15.24" y1="152.4" x2="-15.24" y2="127" width="0.1524" layer="91"/>
 </segment>
 </net>
