File: Rail/pcb1.brd (EAGLE design)
At the start: 0 parts

Commit message: dimension
Other:
- board outline added: 99.4 x 172.8 mm

Commit message: ..
Other:
- board outline removed

Commit message: outline
Parts:
- added J1: (no value), Wurth_Connectors_WR-PHD:61301821121
Other:
- board outline added: 49.7 x 86.4 mm
Changed lines of the file:
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@@
 <setting verticaltext="up"/>
 </settings>
-<grid distance="50" unitdist="mil" unit="mil" style="lines" multiple="1" display="no" altdistance="5" altunitdist="mil" altunit="mil"/>
+<grid distance="50" unitdist="mil" unit="mm" style="lines" multiple="1" display="no" altdistance="5" altunitdist="mil" altunit="mil"/>
 <layers>
 <layer number="1" name="Top" color="4" fill="1" visible="yes" active="yes"/>
@@
 <layer number="48" name="Document" color="7" fill="1" visible="yes" active="yes"/>
 <layer number="49" name="Reference" color="7" fill="1" visible="yes" active="yes"/>
+<layer number="50" name="dxf" color="7" fill="1" visible="no" active="no"/>
 <layer number="51" name="tDocu" color="7" fill="1" visible="yes" active="yes"/>
 <layer number="52" name="bDocu" color="7" fill="1" visible="yes" active="yes"/>
+<layer number="90" name="Modules" color="7" fill="1" visible="no" active="no"/>
+<layer number="91" name="Nets" color="2" fill="1" visible="no" active="no"/>
+<layer number="92" name="Busses" color="1" fill="1" visible="no" active="no"/>
+<layer number="93" name="Pins" color="2" fill="1" visible="no" active="no"/>
+<layer number="94" name="Symbols" color="4" fill="1" visible="no" active="no"/>
+<layer number="95" name="Names" color="7" fill="1" visible="no" active="no"/>
+<layer number="96" name="Values" color="7" fill="1" visible="no" active="no"/>
+<layer number="97" name="Info" color="7" fill="1" visible="no" active="no"/>
+<layer number="98" name="Guide" color="6" fill="1" visible="no" active="no"/>
+<layer number="250" name="Descript" color="7" fill="1" visible="yes" active="yes"/>
+<layer number="251" name="SMDround" color="7" fill="1" visible="yes" active="yes"/>
 </layers>
 <board>
@@
 <wire x1="18.23" y1="-2.54" x2="17.13" y2="-2.54" width="0.001" layer="49"/>
 <wire x1="-24.85" y1="0" x2="8.32553125" y2="0" width="0.001" layer="49"/>
-<wire x1="-15.72633125" y1="43.2" x2="-2.27366875" y2="43.2" width="0.001" layer="49"/>
-<wire x1="-20.263440625" y1="43.2" x2="-15.736559375" y2="43.2" width="0.001" layer="49"/>
-<wire x1="-24.85" y1="43.2" x2="-20.27366875" y2="43.2" width="0.001" layer="49"/>
-<wire x1="-24.85" y1="-43.2" x2="-24.85" y2="-22.7" width="0.001" layer="49"/>
-<wire x1="-24.85" y1="-22.7" x2="-24.85" y2="-22.11243125" width="0.001" layer="49"/>
-<wire x1="-20.27366875" y1="-43.2" x2="-24.85" y2="-43.2" width="0.001" layer="49"/>
-<wire x1="-24.85" y1="22.11243125" x2="-24.85" y2="22.7" width="0.001" layer="49"/>
-<wire x1="-24.85" y1="22.7" x2="-24.85" y2="43.2" width="0.001" layer="49"/>
-<wire x1="-24.1" y1="-20.067359375" x2="-24.1" y2="-0.8" width="0.001" layer="49"/>
-<wire x1="-24.1" y1="0.8" x2="-24.1" y2="20.067359375" width="0.001" layer="49"/>
-<wire x1="-24.1" y1="20.067359375" x2="-24.1" y2="21" width="0.001" layer="49"/>
-<wire x1="-2.27366875" y1="-43.2" x2="-15.72633125" y2="-43.2" width="0.001" layer="49"/>
-<wire x1="-2.263440625" y1="43.2" x2="2.263440625" y2="43.2" width="0.001" layer="49"/>
-<wire x1="24.85" y1="-43.2" x2="20.27366875" y2="-43.2" width="0.001" layer="49"/>
-<wire x1="15.72633125" y1="-43.2" x2="2.27366875" y2="-43.2" width="0.001" layer="49"/>
-<wire x1="-15.736559375" y1="-43.2" x2="-20.263440625" y2="-43.2" width="0.001" layer="49"/>
-<wire x1="20.263440625" y1="-43.2" x2="15.736559375" y2="-43.2" width="0.001" layer="49"/>
+<wire x1="-24.85" y1="-43.2" x2="-24.85" y2="-22.11243125" width="0.001" layer="20"/>
+<wire x1="-24.85" y1="22.11243125" x2="-24.85" y2="43.2" width="0.001" layer="20"/>
+<wire x1="-24.1" y1="-21" x2="-24.1" y2="21" width="0.001" layer="20"/>
 <wire x1="10.361009375" y1="1.0325" x2="11.186009375" y2="0.92" width="0.001" layer="49"/>
 <wire x1="10.398509375" y1="-8.02375" x2="10.642259375" y2="-8.2675" width="0.001" layer="49"/>
@@
 <wire x1="9.686009375" y1="-7.2925" x2="9.686009375" y2="-6.29875" width="0.001" layer="49"/>
 <wire x1="9.798509375" y1="-6.29875" x2="9.929759375" y2="-6.33625" width="0.001" layer="49"/>
-<wire x1="15.736559375" y1="43.2" x2="20.263440625" y2="43.2" width="0.001" layer="49"/>
-<wire x1="2.27366875" y1="43.2" x2="15.72633125" y2="43.2" width="0.001" layer="49"/>
-<wire x1="20.27366875" y1="43.2" x2="24.85" y2="43.2" width="0.001" layer="49"/>
-<wire x1="24.85" y1="43.2" x2="24.85" y2="22.7" width="0.001" layer="49"/>
-<wire x1="24.85" y1="22.7" x2="24.85" y2="22.11243125" width="0.001" layer="49"/>
-<wire x1="24.1" y1="-0.8" x2="24.1" y2="-20.067359375" width="0.001" layer="49"/>
-<wire x1="24.1" y1="21" x2="24.1" y2="20.067359375" width="0.001" layer="49"/>
-<wire x1="24.1" y1="20.067359375" x2="24.1" y2="0.8" width="0.001" layer="49"/>
-<wire x1="-24.1" y1="-21" x2="-24.1" y2="-20.067359375" width="0.001" layer="49"/>
-<wire x1="24.1" y1="-20.067359375" x2="24.1" y2="-21" width="0.001" layer="49"/>
-<wire x1="24.85" y1="-22.11243125" x2="24.85" y2="-22.7" width="0.001" layer="49"/>
-<wire x1="2.263440625" y1="-43.2" x2="-2.263440625" y2="-43.2" width="0.001" layer="49"/>
-<wire x1="24.85" y1="-22.7" x2="24.85" y2="-43.2" width="0.001" layer="49"/>
-<wire x1="-24.1" y1="21" x2="-24.85" y2="22.11243125" width="0.001" layer="49" curve="67.975714"/>
-<wire x1="24.1" y1="-21" x2="24.85" y2="-22.11243125" width="0.001" layer="49" curve="67.975714"/>
-<wire x1="-24.85" y1="-22.11243125" x2="-24.1" y2="-21" width="0.001" layer="49" curve="67.975714"/>
-<wire x1="24.85" y1="22.11243125" x2="24.1" y2="21" width="0.001" layer="49" curve="67.975714"/>
+<wire x1="24.85" y1="43.2" x2="24.85" y2="22.11243125" width="0.001" layer="20"/>
+<wire x1="24.1" y1="21" x2="24.1" y2="-21" width="0.001" layer="20"/>
+<wire x1="24.85" y1="-22.11243125" x2="24.85" y2="-43.2" width="0.001" layer="20"/>
+<wire x1="-24.1" y1="21" x2="-24.85" y2="22.11243125" width="0.001" layer="20" curve="67.975714"/>
+<wire x1="24.1" y1="-21" x2="24.85" y2="-22.11243125" width="0.001" layer="20" curve="67.975714"/>
+<wire x1="-24.85" y1="-22.11243125" x2="-24.1" y2="-21" width="0.001" layer="20" curve="67.975714"/>
+<wire x1="24.85" y1="22.11243125" x2="24.1" y2="21" width="0.001" layer="20" curve="67.975714"/>
 <circle x="17.68" y="-5.08" radius="0.5" width="0.001" layer="49"/>
 <circle x="17.68" y="7.62" radius="0.5" width="0.001" layer="49"/>
@@
 <wire x1="2.45" y1="-20.067359375" x2="2.45" y2="-20.8" width="0.001" layer="49"/>
 <wire x1="2.45" y1="-20.8" x2="-2.45" y2="-20.8" width="0.001" layer="49"/>
-<wire x1="24.1" y1="0.8" x2="24.1" y2="-0.8" width="0.001" layer="49"/>
 <wire x1="24.1" y1="-0.8" x2="23.3" y2="-0.8" width="0.001" layer="49"/>
 <wire x1="23.3" y1="-0.8" x2="23.3" y2="0.8" width="0.001" layer="49"/>
@@
 <wire x1="-23.3" y1="0.8" x2="-23.3" y2="-0.8" width="0.001" layer="49"/>
 <wire x1="-23.3" y1="-0.8" x2="-24.1" y2="-0.8" width="0.001" layer="49"/>
-<wire x1="-24.1" y1="-0.8" x2="-24.1" y2="0.8" width="0.001" layer="49"/>
 <wire x1="-24.1" y1="0.8" x2="-23.3" y2="0.8" width="0.001" layer="49"/>
 <wire x1="24.1" y1="20.067359375" x2="20.45" y2="20.067359375" width="0.001" layer="49"/>
@@
 <wire x1="-20.45" y1="20.067359375" x2="-24.1" y2="20.067359375" width="0.001" layer="49"/>
 <wire x1="-24.85" y1="22.7" x2="24.85" y2="22.7" width="0.001" layer="49"/>
+<wire x1="-24.85" y1="-43.2" x2="24.85" y2="-43.2" width="0.001" layer="20"/>
+<wire x1="-24.85" y1="43.2" x2="24.85" y2="43.2" width="0.001" layer="20"/>
 </plain>
 <attributes>
@@
 </autorouter>
 <elements>
+<element name="J1" library="Wurth_Connectors_WR-PHD" library_urn="urn:adsk.eagle:library:14804658" package="61301821121" package3d_urn="urn:adsk.eagle:package:14805433/2" value="" x="18.95" y="0" smashed="yes" rot="R90">
+<attribute name="DATASHEET-URL" value="https://katalog.we-online.com/em/datasheet/61301821121.pdf" x="18.95" y="0" size="1.778" layer="27" font="vector" rot="R90" display="off"/>
+<attribute name="GENDER" value="Pin Header" x="18.95" y="0" size="1.778" layer="27" font="vector" rot="R90" display="off"/>
+<attribute name="IR" value="3A" x="18.95" y="0" size="1.778" layer="27" font="vector" rot="R90" display="off"/>
+<attribute name="MATES" value="WR-PHD 2.54mm Angled DualSocket Header/Dual Socket Header/Dual Socket Header Bottom Entry/Dual Socket Header Bottom Entry Large/SMT Dual Socket Header/SMT Dual Socket Header Bottom Entry" x="18.95" y="0" size="1.778" layer="27" font="vector" rot="R90" display="off"/>
+<attribute name="NAME" x="18.1939" y="-12.3276" size="0.8128" layer="25" rot="R90" align="bottom-right"/>
+<attribute name="PACKAGING" value="Bag" x="18.95" y="0" size="1.778" layer="27" font="vector" rot="R90" display="off"/>
+<attribute name="PART-NUMBER" value=" 61301821121 " x="18.95" y="0" size="1.778" layer="27" font="vector" rot="R90" display="off"/>
+<attribute name="PINS" value=" 18 " x="18.95" y="0" size="1.778" layer="27" font="vector" rot="R90" display="off"/>
+<attribute name="ROWS" value="Dual" x="18.95" y="0" size="1.778" layer="27" font="vector" rot="R90" display="off"/>
+<attribute name="TYPE" value="Board Stacker" x="18.95" y="0" size="1.778" layer="27" font="vector" rot="R90" display="off"/>
+<attribute name="VALUE" x="19.8942" y="-12.2476" size="0.8128" layer="27" rot="R90" align="bottom-right"/>
+</element>
 </elements>
 <signals>
@@
 </board>
 </drawing>
+<compatibility>
+<note version="8.2" severity="warning">
+Since Version 8.2, EAGLE supports online libraries. The ids
+of those online libraries will not be understood (or retained)
+with this version.
+</note>
+<note version="8.3" severity="warning">
+Since Version 8.3, EAGLE supports URNs for individual library
+assets (packages, symbols, and devices). The URNs of those assets
+will not be understood (or retained) with this version.
+</note>
+<note version="8.3" severity="warning">
+Since Version 8.3, EAGLE supports the association of 3D packages
+with devices in libraries, schematics, and board files. Those 3D
+packages will not be understood (or retained) with this version.
+</note>
+</compatibility>
 </eagle>

Commit message: not finished. ..
Parts:
- flipped J1 to the bottom

Commit message: ..
Parts:
- added C1: 47uF, Wurth_Capacitors_WCAP-CSGP:WCAP-CSGP_1210_H2.5
- added C15: 47 nF, fliegl-wuerth:WCAP-CSGP_0402
- added C17, C19: 100 nF, fliegl-wuerth:WCAP-CSGP_0402
- added D1: 26V, Wurth_EMC Components_WE-TVSP:WE-TVSP_DO-214AC_BIDIRECTIONAL
- added D3: SS12L_R3, SS12L_R3:SODFL3618X143N
- added D6: 26.2V / 35pF, fliegl-wuerth:WE-TVS_SOT23-3L
- added J2: (no value), Wurth_Connectors_WR-PHD:61300411121
- added J3: (no value), Wurth_Connectors_WR-PHD:61300511121
- added R21, R22: 60.4R 1%, Resistor_smaller_fliegl:WCAP-CSRF_0402
- added U1: (no value), Wurth_Step Down Converter_MagI³C-FDSM:MAGI³C-FDSM_173XXXX42
- added U4: TLE9250VSJ, TLE9250VSJ:SOIC127P602X173-8N-V
- added X1: S4P-VH, con-JST VH:S4P-VH
- moved J1 37.9 mm to (-18.9, 0.00), turned to 270 degrees
Connections:
- new net +12V: D1.2, D3.2, X1.2
- new net +3V3: C19.1, J3.5, U4.5
- new net +5V: C17.1, J2.2, U1.3, U4.3
- new net CAN1_RXD: J3.4, U4.4
- new net CAN1_TXD: J2.4, U4.1
- new net CAN_H: D6.2, R22.2, U4.7, X1.3
- new net CAN_L: D6.1, R21.1, U4.6, X1.4
- new net GND: C1.1, C15.2, C17.2, C19.2, D1.1, D6.3, J2.1, U1.2, U4.2, U4.8, X1.1
- new net N$1: C1.2, D3.1, U1.1
- new net N$17: C15.1, R21.2, R22.1
Routing:
- added copper zone on layer 1, net GND
- added copper zone on layer 16, net GND
Other:
- board text added: "3V3"
- board text added: "5V"
- board text added: "G"
- board text added: "G19"
- board text added: "G21"
- board text added: "G22"
- board text added: "G23"
- board text added: "G25"
- board text added: "G33"
- board text added: "GND"
- board text added: "H"
- board text added: "L"
- board text added: "V"

Commit message: ..
Parts:
- added C2, C3, C4, C5, C6, C7, C8, C9: 100 nF, Wurth_Capacitors_WCAP-CSGP:WCAP-CSGP_0402
- added J6, J7: 638207222005, Wurth_Connectors_WR-FAST:638207222005
- added R1, R11: 1k2, Resistor_smaller_fliegl:WCAP-CSRF_0402@1
- added R10, R7: 47R, Resistor_smaller_fliegl:WCAP-CSRF_0402@1
- added R12, R13, R15, R16, R18, R2, R3, R4, R5, R6: 4k7, Resistor_smaller_fliegl:WCAP-CSRF_0402@1
- added R14, R17, R8, R9: 47k, Resistor_smaller_fliegl:WCAP-CSRF_0402@1
- added U2, U3: (no value), BTS7030-2EPA:SOP65P600X115-15N-V
- moved U1 94.6 mm to (42.3, 52.8)
- moved X1 70.6 mm to (16.9, 35.5)
- moved C15 67.0 mm to (13.1, 14.5)
- moved R21 67.0 mm to (11.8, 14.5)
- moved R22 67.0 mm to (14.3, 14.5)
- moved D6 66.9 mm to (13.0, 18.0)
- moved C17 48.3 mm to (-9.22, 15.3), turned to 0 degrees
- moved U4 45.6 mm to (-9.13, 10.6), turned to 270 degrees
- moved C19 41.8 mm to (-10.5, 5.87), turned to 0 degrees
Connections:
- new net AGNDU2: C6.2, R10.2, U2.1
- new net AGNDU3: C3.2, R7.2, U3.1
- new net DENU2: R16.1
- new net DENU3: R6.1
- new net DSELU2: R12.1
- new net DSELU3: R3.1
- new net ISOU2: R11.2, R15.2, U2.4
- new net ISOU3: R1.2, R5.2, U3.4
- new net ISU2: R15.1
- new net ISU3: R5.1
- new net N$10: R18.2, U2.2
- new net N$13: R12.2, U2.5
- new net N$14: R13.2, U2.6
- new net N$15: R16.2, U2.3
- new net N$2: R2.2, U3.2
- new net N$3: R3.2, U3.5
- new net N$4: R4.2, U3.6
- new net N$5: R6.2, U3.3
- new net N$6: J6.5, J6.A5
- new net Q1: C7.2, J7.2, J7.A2, R14.2, U2.10, U2.8, U2.9
- new net Q1C: J3.3, R13.1
- new net Q2: C8.1, J7.3, J7.A3, R17.1, U2.12, U2.13, U2.14
- new net Q2C: J3.2, R18.1
- new net Q3: C4.2, J7.4, J7.A4, R9.2, U3.10, U3.8, U3.9
- new net Q3C: J3.1, R4.1
- new net Q4: C9.1, J7.5, J7.A5, R8.1, U3.12, U3.13, U3.14
- new net Q4C: J2.3, R2.1
- net +12V: now also C2.1, C3.1, C5.1, C6.1, J7.1, J7.A1, U2.15, U3.15
- net GND: now also C2.2, C4.1, C5.2, C7.1, C8.2, C9.2, R1.1, R10.1, R11.1, R14.1, R17.2, R7.1, R8.2, R9.1
Routing:
- net Q3C: track 0.00 -> 66.3 mm, vias 0 -> 1
- net Q2C: track 0.00 -> 60.7 mm, vias 0 -> 1
- net Q1C: track 0.00 -> 57.0 mm, vias 0 -> 1
- net Q4C: track 0.00 -> 56.0 mm, vias 0 -> 1
- net CAN_H: track 0.00 -> 50.4 mm
- net CAN_L: track 0.00 -> 48.6 mm
- net +5V: track 0.00 -> 28.5 mm
- net CAN1_RXD: track 0.00 -> 25.0 mm
- net CAN1_TXD: track 0.00 -> 22.3 mm
- net ISOU3: track 0.00 -> 7.37 mm
- net ISOU2: track 0.00 -> 7.37 mm
- net N$5: track 0.00 -> 4.52 mm
- net N$3: track 0.00 -> 4.52 mm
- net N$15: track 0.00 -> 4.52 mm
- net N$13: track 0.00 -> 4.52 mm
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- added copper zone on layer 1, net +12V
- added copper zone on layer 1, net Q1
- added copper zone on layer 1, net Q2
- added copper zone on layer 1, net Q3
- added copper zone on layer 1, net Q4
- removed copper zone on layer 1, net GND
- removed copper zone on layer 16, net GND
Other:
- board text added: "Q1"
- board text added: "Q2"
- board text added: "Q3"
- board text added: "Q4"
- board text removed: "G"
- board text removed: "H"
- board text removed: "L"
- board text removed: "V"

Commit message: ..
Parts:
- removed C1: 47uF, Wurth_Capacitors_WCAP-CSGP:WCAP-CSGP_1210_H2.5
- removed D3: SS12L_R3, SS12L_R3:SODFL3618X143N
- removed U1: (no value), Wurth_Step Down Converter_MagI³C-FDSM:MAGI³C-FDSM_173XXXX42
- added C10: 47uF, Wurth_Capacitors_WCAP-CSGP:WCAP-CSGP_1210_H2.5
- added C11: 100 nF, fliegl-wuerth:WCAP-CSGP_0402
- added C12: 22 µF, Wurth_Capacitors_WCAP-CSGP:WCAP-CSGP_0805_H1.25_R
- added D2: 26V, Wurth_EMC Components_WE-TVSP:WE-TVSP_DO-214AC_BIDIRECTIONAL
- added G1: TLE4270-2D-INF-PG-TO252-5-11_L_1, INF-PG-TO252-5-11L:INF-PG-TO252-5-11_L_1PRIMARY
- D1: value 26V -> 33V; device Wurth_EMC Components_WE-TVSP:WE-TVSP_DO-214AC_BIDIRECTIONAL -> Wurth_EMC Components_WE-TVSP:WE-TVSP_DO-214AB_BIDIRECTIONAL
- moved D1 78.1 mm to (0.20, -9.86), turned to 0 degrees
- moved C7 40.3 mm to (6.35, -16.5), turned to 180 degrees
- moved C8 31.1 mm to (14.0, -16.5), turned to 180 degrees
- moved R14 29.3 mm to (6.35, -17.8), turned to 180 degrees
- moved R17 28.3 mm to (14.0, -17.8), turned to 180 degrees
- moved C4 14.1 mm to (16.5, -17.8), turned to 180 degrees
- moved R8 13.7 mm to (22.9, -16.5), turned to 180 degrees
- moved R9 12.6 mm to (16.5, -16.5), turned to 180 degrees
- moved C9 10.7 mm to (22.9, -17.8), turned to 180 degrees
- moved R13 2.54 mm to (8.86, -5.79)
- moved R18 2.54 mm to (11.5, -5.79)
- moved R2 2.54 mm to (21.6, -5.79)
- moved R4 2.54 mm to (19.0, -5.79)
- moved U2 2.54 mm to (10.2, -11.4)
- moved U3 2.54 mm to (20.3, -11.4)
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Connections:
- removed net N$1: C1.2, D3.1, U1.1
- new net +12V1: C10.2, D2.2, G1.1, X1.2
- new net N$7: C11.1, G1.4
- net +12V: no longer D3.2, X1.2
- net +5V: now also C12.2, G1.5; no longer U1.3
- net GND: now also C10.1, C11.2, C12.1, D2.1, G1.3; no longer C1.1, U1.2
Routing:
- net +3V3: track 2.01 -> 32.1 mm
- net Q4C: track 56.0 -> 50.1 mm, vias 1 -> 0
- net Q3C: track 66.3 -> 63.8 mm, vias 1 -> 0
- net Q2C: track 60.7 -> 58.1 mm, vias 1 -> 0
- net Q1C: track 57.0 -> 54.5 mm, vias 1 -> 0
- added copper zone on layer 1, net +12V1

Commit message: ..
Routing:
- added copper zone on layer 1, net GND
Changed lines of the file:
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@@
 <drawing>
 <settings>
-<setting alwaysvectorfont="no"/>
+<setting alwaysvectorfont="yes"/>
 <setting verticaltext="up"/>
 </settings>
@@
 <contactref element="C12" pad="1"/>
 <contactref element="D1" pad="1"/>
-<wire x1="22.42" y1="17.8816" x2="22.87" y2="35.5" width="0" layer="19" extent="1-1"/>
-<wire x1="22.886" y1="14.0208" x2="22.42" y2="17.8816" width="0" layer="19" extent="1-1"/>
-<wire x1="12.97" y1="19.09" x2="22.42" y2="17.8816" width="0" layer="19" extent="1-1"/>
-<wire x1="13.0504" y1="14.0146" x2="12.97" y2="19.09" width="0" layer="19" extent="1-1"/>
-<wire x1="14.4352" y1="12.0396" x2="13.0504" y2="14.0146" width="0" layer="19" extent="1-1"/>
-<wire x1="10.16" y1="-0.2112" x2="14.4352" y2="12.0396" width="0" layer="19" extent="1-1"/>
+<polygon width="0.2032" layer="1" thermals="no" rank="2">
+<vertex x="-50.4168" y="0"/>
+<vertex x="-50.4168" y="51.451"/>
+<vertex x="57.2168" y="51.451"/>
+<vertex x="57.2168" y="0"/>
+</polygon>
+<wire x1="22.27" y1="-3.056" x2="23.0424" y2="-5.2728" width="0" layer="19" extent="1-1"/>
+<wire x1="20.32" y1="1.9732" x2="22.27" y2="-3.056" width="0" layer="19" extent="1-1"/>
 <wire x1="12.11" y1="-3.056" x2="10.16" y2="-0.2112" width="0" layer="19" extent="1-1"/>
 <wire x1="12.7928" y1="-5.2912" x2="12.11" y2="-3.056" width="0" layer="19" extent="1-1"/>
-<wire x1="16.6056" y1="3.3752" x2="14.4352" y2="12.0396" width="0" layer="19" extent="1-1"/>
-<wire x1="11.932" y1="8.6864" x2="16.6056" y2="3.3752" width="0" layer="19" extent="1-1"/>
-<wire x1="20.32" y1="1.9732" x2="11.932" y2="8.6864" width="0" layer="19" extent="1-1"/>
-<wire x1="22.27" y1="-3.056" x2="20.32" y2="1.9732" width="0" layer="19" extent="1-1"/>
-<wire x1="23.0424" y1="-5.2728" x2="22.27" y2="-3.056" width="0" layer="19" extent="1-1"/>
 <wire x1="23.36" y1="-16.51" x2="23.0424" y2="-5.2728" width="0" layer="19" extent="1-1"/>
 <wire x1="23.36" y1="-17.78" x2="23.36" y2="-16.51" width="0" layer="19" extent="1-1"/>
@@
 <wire x1="5.85" y1="-16.51" x2="5.85" y2="-17.78" width="0" layer="19" extent="1-1"/>
 <wire x1="-3.2968" y1="-9.8552" x2="5.85" y2="-16.51" width="0" layer="19" extent="1-1"/>
-<wire x1="-9.9654" y1="5.8726" x2="-3.2968" y2="-9.8552" width="0" layer="19" extent="1-1"/>
-<wire x1="-7.2226" y1="7.8574" x2="-9.9654" y2="5.8726" width="0" layer="19" extent="1-1"/>
-<wire x1="-8.4926" y1="13.3874" x2="-7.2226" y2="7.8574" width="0" layer="19" extent="1-1"/>
-<wire x1="-8.7178" y1="15.311" x2="-8.4926" y2="13.3874" width="0" layer="19" extent="1-1"/>
-<wire x1="-4.78" y1="42.32" x2="-8.7178" y2="15.311" width="0" layer="19" extent="1-1"/>
 </signal>
 <signal name="+5V">
@@
 <contactref element="C12" pad="2"/>
 <wire x1="11.932" y1="10.5864" x2="14.3256" y2="10.3752" width="0" layer="19" extent="1-1"/>
-<wire x1="-9.7626" y1="13.3874" x2="14.3256" y2="10.3752" width="0" layer="19" extent="1-1"/>
+<wire x1="-9.7626" y1="13.3874" x2="11.932" y2="10.5864" width="0" layer="19" extent="1-1"/>
 <wire x1="-9.7178" y1="15.311" x2="-9.7626" y2="13.3874" width="0" layer="19" extent="1-1"/>
 </signal>
