File: Rail/pcb1.brd (EAGLE design)
At the start: 49.7 x 86.4 mm, 45 parts, among them J6 638207222005, J7 638207222005, U4 TLE9250VSJ, X1 S4P-VH

Commit message: LED and Resisotr !
Parts:
- RX1, RX2, RX3, RX4: value 470Ohm -> 510mOhm; device Wurth_Resistor_WRIS-KWKB:WRIS-KWKB_0612 -> Wurth_Resistor_WRIS-KWKH:WRIS-KWKH_0612
Changed lines of the file:
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@@
 <drawing>
 <settings>
-<setting alwaysvectorfont="yes"/>
+<setting alwaysvectorfont="no"/>
 <setting verticaltext="up"/>
 </settings>
@@
 <attribute name="VCLAMP" value="53.3V" x="-20.066" y="-26.035" size="1.778" layer="27" display="off"/>
 </element>
-<element name="RX4" library="Wurth_Resistor_WRIS-KWKB" library_urn="urn:adsk.eagle:library:13351500" package="WRIS-KWKB_0612" package3d_urn="urn:adsk.eagle:package:13351506/2" value="470Ohm" x="23.495" y="-25.4" smashed="yes" rot="R90">
-<attribute name="DATASHEET-URL" value="https://katalog.we-online.de/pbs/datasheet/561020132023.pdf" x="23.495" y="-25.4" size="1.778" layer="27" rot="R90" display="off"/>
-<attribute name="IR" value="39.9mA" x="23.495" y="-25.4" size="1.778" layer="27" rot="R90" display="off"/>
+<element name="RX4" library="Wurth_Resistor_WRIS-KWKH" library_urn="urn:adsk.eagle:library:13353576" package="WRIS-KWKH_0612" package3d_urn="urn:adsk.eagle:package:13353581/2" value="510mOhm" x="23.495" y="-25.4" smashed="yes" rot="R90">
+<attribute name="DATASHEET-URL" value="https://katalog.we-online.de/pbs/datasheet/561070332078.pdf" x="23.495" y="-25.4" size="1.778" layer="27" rot="R90" display="off"/>
+<attribute name="IR" value="1.4A" x="23.495" y="-25.4" size="1.778" layer="27" rot="R90" display="off"/>
 <attribute name="MOUNT" value="SMT" x="23.495" y="-25.4" size="1.778" layer="27" rot="R90" display="off"/>
 <attribute name="NAME" x="23.495" y="-23.7" size="0.8128" layer="25" align="bottom-center"/>
-<attribute name="PART-NUMBER" value=" 561020132023 " x="23.495" y="-25.4" size="1.778" layer="27" rot="R90" display="off"/>
-<attribute name="PRATED" value="0.75W" x="23.495" y="-25.4" size="1.778" layer="27" rot="R90" display="off"/>
-<attribute name="TCR" value="±200ppm/ °C" x="23.495" y="-25.4" size="1.778" layer="27" rot="R90" display="off"/>
-<attribute name="TECHNICAL-REFERENCE" value="KB06124700J304DAATP0000" x="23.495" y="-25.4" size="1.778" layer="27" rot="R90" display="off"/>
-</element>
-<element name="RX2" library="Wurth_Resistor_WRIS-KWKB" library_urn="urn:adsk.eagle:library:13351500" package="WRIS-KWKB_0612" package3d_urn="urn:adsk.eagle:package:13351506/2" value="470Ohm" x="3.175" y="-25.4" smashed="yes" rot="R90">
-<attribute name="DATASHEET-URL" value="https://katalog.we-online.de/pbs/datasheet/561020132023.pdf" x="3.175" y="-25.4" size="1.778" layer="27" rot="R90" display="off"/>
-<attribute name="IR" value="39.9mA" x="3.175" y="-25.4" size="1.778" layer="27" rot="R90" display="off"/>
+<attribute name="PART-NUMBER" value=" 561070332078 " x="23.495" y="-25.4" size="1.778" layer="27" rot="R90" display="off"/>
+<attribute name="PRATED" value="1W" x="23.495" y="-25.4" size="1.778" layer="27" rot="R90" display="off"/>
+<attribute name="TCR" value="200ppm/ °C" x="23.495" y="-25.4" size="1.778" layer="27" rot="R90" display="off"/>
+<attribute name="TECHNICAL-REFERENCE" value="KH0612R510F101HAATP0000" x="23.495" y="-25.4" size="1.778" layer="27" rot="R90" display="off"/>
+</element>
+<element name="RX2" library="Wurth_Resistor_WRIS-KWKH" library_urn="urn:adsk.eagle:library:13353576" package="WRIS-KWKH_0612" package3d_urn="urn:adsk.eagle:package:13353581/2" value="510mOhm" x="3.175" y="-25.4" smashed="yes" rot="R90">
+<attribute name="DATASHEET-URL" value="https://katalog.we-online.de/pbs/datasheet/561070332078.pdf" x="3.175" y="-25.4" size="1.778" layer="27" rot="R90" display="off"/>
+<attribute name="IR" value="1.4A" x="3.175" y="-25.4" size="1.778" layer="27" rot="R90" display="off"/>
 <attribute name="MOUNT" value="SMT" x="3.175" y="-25.4" size="1.778" layer="27" rot="R90" display="off"/>
 <attribute name="NAME" x="3.175" y="-23.7" size="0.8128" layer="25" align="bottom-center"/>
-<attribute name="PART-NUMBER" value=" 561020132023 " x="3.175" y="-25.4" size="1.778" layer="27" rot="R90" display="off"/>
-<attribute name="PRATED" value="0.75W" x="3.175" y="-25.4" size="1.778" layer="27" rot="R90" display="off"/>
-<attribute name="TCR" value="±200ppm/ °C" x="3.175" y="-25.4" size="1.778" layer="27" rot="R90" display="off"/>
-<attribute name="TECHNICAL-REFERENCE" value="KB06124700J304DAATP0000" x="3.175" y="-25.4" size="1.778" layer="27" rot="R90" display="off"/>
-</element>
-<element name="RX1" library="Wurth_Resistor_WRIS-KWKB" library_urn="urn:adsk.eagle:library:13351500" package="WRIS-KWKB_0612" package3d_urn="urn:adsk.eagle:package:13351506/2" value="470Ohm" x="-13.335" y="-25.4" smashed="yes" rot="R90">
-<attribute name="DATASHEET-URL" value="https://katalog.we-online.de/pbs/datasheet/561020132023.pdf" x="-13.335" y="-25.4" size="1.778" layer="27" rot="R90" display="off"/>
-<attribute name="IR" value="39.9mA" x="-13.335" y="-25.4" size="1.778" layer="27" rot="R90" display="off"/>
+<attribute name="PART-NUMBER" value=" 561070332078 " x="3.175" y="-25.4" size="1.778" layer="27" rot="R90" display="off"/>
+<attribute name="PRATED" value="1W" x="3.175" y="-25.4" size="1.778" layer="27" rot="R90" display="off"/>
+<attribute name="TCR" value="200ppm/ °C" x="3.175" y="-25.4" size="1.778" layer="27" rot="R90" display="off"/>
+<attribute name="TECHNICAL-REFERENCE" value="KH0612R510F101HAATP0000" x="3.175" y="-25.4" size="1.778" layer="27" rot="R90" display="off"/>
+</element>
+<element name="RX1" library="Wurth_Resistor_WRIS-KWKH" library_urn="urn:adsk.eagle:library:13353576" package="WRIS-KWKH_0612" package3d_urn="urn:adsk.eagle:package:13353581/2" value="510mOhm" x="-13.335" y="-25.4" smashed="yes" rot="R90">
+<attribute name="DATASHEET-URL" value="https://katalog.we-online.de/pbs/datasheet/561070332078.pdf" x="-13.335" y="-25.4" size="1.778" layer="27" rot="R90" display="off"/>
+<attribute name="IR" value="1.4A" x="-13.335" y="-25.4" size="1.778" layer="27" rot="R90" display="off"/>
 <attribute name="MOUNT" value="SMT" x="-13.335" y="-25.4" size="1.778" layer="27" rot="R90" display="off"/>
 <attribute name="NAME" x="-13.335" y="-23.7" size="0.8128" layer="25" align="bottom-center"/>
-<attribute name="PART-NUMBER" value=" 561020132023 " x="-13.335" y="-25.4" size="1.778" layer="27" rot="R90" display="off"/>
-<attribute name="PRATED" value="0.75W" x="-13.335" y="-25.4" size="1.778" layer="27" rot="R90" display="off"/>
-<attribute name="TCR" value="±200ppm/ °C" x="-13.335" y="-25.4" size="1.778" layer="27" rot="R90" display="off"/>
-<attribute name="TECHNICAL-REFERENCE" value="KB06124700J304DAATP0000" x="-13.335" y="-25.4" size="1.778" layer="27" rot="R90" display="off"/>
-</element>
-<element name="RX3" library="Wurth_Resistor_WRIS-KWKB" library_urn="urn:adsk.eagle:library:13351500" package="WRIS-KWKB_0612" package3d_urn="urn:adsk.eagle:package:13351506/2" value="470Ohm" x="6.985" y="-25.4" smashed="yes" rot="R90">
-<attribute name="DATASHEET-URL" value="https://katalog.we-online.de/pbs/datasheet/561020132023.pdf" x="6.985" y="-25.4" size="1.778" layer="27" rot="R90" display="off"/>
-<attribute name="IR" value="39.9mA" x="6.985" y="-25.4" size="1.778" layer="27" rot="R90" display="off"/>
+<attribute name="PART-NUMBER" value=" 561070332078 " x="-13.335" y="-25.4" size="1.778" layer="27" rot="R90" display="off"/>
+<attribute name="PRATED" value="1W" x="-13.335" y="-25.4" size="1.778" layer="27" rot="R90" display="off"/>
+<attribute name="TCR" value="200ppm/ °C" x="-13.335" y="-25.4" size="1.778" layer="27" rot="R90" display="off"/>
+<attribute name="TECHNICAL-REFERENCE" value="KH0612R510F101HAATP0000" x="-13.335" y="-25.4" size="1.778" layer="27" rot="R90" display="off"/>
+</element>
+<element name="RX3" library="Wurth_Resistor_WRIS-KWKH" library_urn="urn:adsk.eagle:library:13353576" package="WRIS-KWKH_0612" package3d_urn="urn:adsk.eagle:package:13353581/2" value="510mOhm" x="6.985" y="-25.4" smashed="yes" rot="R90">
+<attribute name="DATASHEET-URL" value="https://katalog.we-online.de/pbs/datasheet/561070332078.pdf" x="6.985" y="-25.4" size="1.778" layer="27" rot="R90" display="off"/>
+<attribute name="IR" value="1.4A" x="6.985" y="-25.4" size="1.778" layer="27" rot="R90" display="off"/>
 <attribute name="MOUNT" value="SMT" x="6.985" y="-25.4" size="1.778" layer="27" rot="R90" display="off"/>
 <attribute name="NAME" x="6.985" y="-23.7" size="0.8128" layer="25" align="bottom-center"/>
-<attribute name="PART-NUMBER" value=" 561020132023 " x="6.985" y="-25.4" size="1.778" layer="27" rot="R90" display="off"/>
-<attribute name="PRATED" value="0.75W" x="6.985" y="-25.4" size="1.778" layer="27" rot="R90" display="off"/>
-<attribute name="TCR" value="±200ppm/ °C" x="6.985" y="-25.4" size="1.778" layer="27" rot="R90" display="off"/>
-<attribute name="TECHNICAL-REFERENCE" value="KB06124700J304DAATP0000" x="6.985" y="-25.4" size="1.778" layer="27" rot="R90" display="off"/>
+<attribute name="PART-NUMBER" value=" 561070332078 " x="6.985" y="-25.4" size="1.778" layer="27" rot="R90" display="off"/>
+<attribute name="PRATED" value="1W" x="6.985" y="-25.4" size="1.778" layer="27" rot="R90" display="off"/>
+<attribute name="TCR" value="200ppm/ °C" x="6.985" y="-25.4" size="1.778" layer="27" rot="R90" display="off"/>
+<attribute name="TECHNICAL-REFERENCE" value="KH0612R510F101HAATP0000" x="6.985" y="-25.4" size="1.778" layer="27" rot="R90" display="off"/>
 </element>
 <element name="D5" library="Wurth_EMC Components_WE-TVSP" library_urn="urn:adsk.eagle:library:14283044" package="WE-TVSP_DO-214AB_BIDIRECTIONAL" package3d_urn="urn:adsk.eagle:package:12146529/2" value="33V" x="20.066" y="26.035" smashed="yes" rot="R180">
@@
 </polygon>
 <contactref element="D2" pad="1"/>
-<wire x1="0.48" y1="-25.4" x2="2.425" y2="-25.4" width="0" layer="19" extent="1-1"/>
 </signal>
 <signal name="N$8" class="1">
@@
 </polygon>
 <contactref element="D1" pad="1"/>
-<wire x1="-10.64" y1="-25.4" x2="-12.585" y2="-25.4" width="0" layer="19" extent="1-1"/>
 </signal>
 <signal name="N$9" class="1">
@@
 </polygon>
 <contactref element="D3" pad="1"/>
-<wire x1="9.68" y1="-25.4" x2="7.735" y2="-25.4" width="0" layer="19" extent="1-1"/>
 </signal>
 <signal name="PWR_GND">
