File: Rail/pcb1.sch (EAGLE design)
At the start: 1 part

Commit message: ..
Parts:
- added C1: 47uF, Wurth_Capacitors_WCAP-CSGP:WCAP-CSGP_1210_H2.5_885012109014_25V(DC)
- added C15: 47 nF, fliegl-wuerth:WCAP-CSGP_0402_885012205054_25V(DC)
- added C17, C19: 100 nF, fliegl-wuerth:WCAP-CSGP_0402_885012205037_16V(DC)
- added D1: 26V, Wurth_EMC Components_WE-TVSP:WE-TVSP_DO-214AC_400W_BI_824501261
- added D3: SS12L_R3, SS12L_R3:SS12L_R3
- added D6: 26.2V / 35pF, fliegl-wuerth:WE-TVS_SOT23-3L_824098024
- added J2: (no value), Wurth_Connectors_WR-PHD:6130XX11121_61300411121
- added J3: (no value), Wurth_Connectors_WR-PHD:6130XX11121_61300511121
- added R21, R22: 60.4R 1%, Resistor_smaller_fliegl:R-0402_60.4OHMS_1%_AEC-Q200
- added U1: (no value), Wurth_Step Down Converter_MagI³C-FDSM:MAGI³C-FDSM_SIP-3_173010542_173XXXX42
- added U4: TLE9250VSJ, TLE9250VSJ:TLE9250VSJ
- added X1: S4P-VH, con-JST VH:S4P-VH
Connections:
- new net +12V: D1.2, D3.A, X1.2
- new net +3V3: C19.1, J3.5, U4.VIO
- new net +5V: C17.1, J2.2, U1.VOUT, U4.VCC
- new net CAN1_RXD: J3.4, U4.RXD
- new net CAN1_TXD: J2.4, U4.TXD
- new net CAN_H: D6.2, R22.2, U4.CANH, X1.3
- new net CAN_L: D6.1, R21.1, U4.CANL, X1.4
- new net GND: C1.1, C15.2, C17.2, C19.2, D1.1, D6.3, J2.1, U1.GND, U4.GND, U4.NEN, X1.1
- new net N$1: C1.2, D3.K, U1.VIN
- new net N$17: C15.1, R21.2, R22.1
Other:
- note added: "3V3"
- note added: "5V"
- note added: "G"
- note added: "G19"
- note added: "G21"
- note added: "G22"
- note added: "G23"
- note added: "G25"
- note added: "G33"
- note added: "GND"
- note added: "H"
- note added: "L"
- note added: "V"
- note added: "Very low electromagnetic emission (EME) allows the use without additional common mode choke TLE9250VSJ"

Commit message: ..
Parts:
- added C2, C3, C4, C5, C6, C7, C8, C9: 100 nF, Wurth_Capacitors_WCAP-CSGP:WCAP-CSGP_0402_885012205086_50V(DC)
- added J6, J7: 638207222005, Wurth_Connectors_WR-FAST:638207222005
- added R1, R11: 1k2, Resistor_smaller_fliegl:R-EU_WCAP-CSGP_0402
- added R10, R7: 47R, Resistor_smaller_fliegl:R-EU_WCAP-CSGP_0402
- added R12, R13, R15, R16, R18, R2, R3, R4, R5, R6: 4k7, Resistor_smaller_fliegl:R-EU_WCAP-CSGP_0402
- added R14, R17, R8, R9: 47k, Resistor_smaller_fliegl:R-EU_WCAP-CSGP_0402
- added U2, U3: (no value), BTS7030-2EPA:BTS7030-2EPA
Connections:
- new net AGNDU2: C6.2, R10.2, U2.GND
- new net AGNDU3: C3.2, R7.2, U3.GND
- new net DENU2: R16.1
- new net DENU3: R6.1
- new net DSELU2: R12.1
- new net DSELU3: R3.1
- new net ISOU2: R11.2, R15.2, U2.IS
- new net ISOU3: R1.2, R5.2, U3.IS
- new net ISU2: R15.1
- new net ISU3: R5.1
- new net N$10: R18.2, U2.IN0
- new net N$13: R12.2, U2.DSEL
- new net N$14: R13.2, U2.IN1
- new net N$15: R16.2, U2.DEN
- new net N$2: R2.2, U3.IN0
- new net N$3: R3.2, U3.DSEL
- new net N$4: R4.2, U3.IN1
- new net N$5: R6.2, U3.DEN
- new net N$6: J6.5
- new net Q1: C7.2, J7.2, R14.2, U2.OUT1A, U2.OUT1B, U2.OUT1C
- new net Q1C: J3.3, R13.1
- new net Q2: C8.1, J7.3, R17.1, U2.OUT0A, U2.OUT0B, U2.OUT0C
- new net Q2C: J3.2, R18.1
- new net Q3: C4.2, J7.4, R9.2, U3.OUT1A, U3.OUT1B, U3.OUT1C
- new net Q3C: J3.1, R4.1
- new net Q4: C9.1, J7.5, R8.1, U3.OUT0A, U3.OUT0B, U3.OUT0C
- new net Q4C: J2.3, R2.1
- net +12V: now also C2.1, C3.1, C5.1, C6.1, J7.1, U2.VS, U3.VS
- net GND: now also C2.2, C4.1, C5.2, C7.1, C8.2, C9.2, R1.1, R10.1, R11.1, R14.1, R17.2, R7.1, R8.2, R9.1

Commit message: ..
Parts:
- removed C1: 47uF, Wurth_Capacitors_WCAP-CSGP:WCAP-CSGP_1210_H2.5_885012109014_25V(DC)
- removed D3: SS12L_R3, SS12L_R3:SS12L_R3
- removed U1: (no value), Wurth_Step Down Converter_MagI³C-FDSM:MAGI³C-FDSM_SIP-3_173010542_173XXXX42
- added C10: 47uF, Wurth_Capacitors_WCAP-CSGP:WCAP-CSGP_1210_H2.5_885012109014_25V(DC)
- added C11: 100 nF, fliegl-wuerth:WCAP-CSGP_0402_885012205037_16V(DC)
- added C12: 22 µF, Wurth_Capacitors_WCAP-CSGP:WCAP-CSGP_0805_H1.25_885012107011_10V(DC)
- added D2: 26V, Wurth_EMC Components_WE-TVSP:WE-TVSP_DO-214AC_400W_BI_824501261
- added G1: TLE4270-2D-INF-PG-TO252-5-11_L_1, INF-PG-TO252-5-11L:TLE4270-2D-INF-PG-TO252-5-11_L_1
- D1: value 26V -> 33V; device Wurth_EMC Components_WE-TVSP:WE-TVSP_DO-214AC_400W_BI_824501261 -> Wurth_EMC Components_WE-TVSP:WE-TVSP_DO-214AB_3000W_BI_824551331
Connections:
- removed net N$1: C1.2, D3.K, U1.VIN
- new net +12V1: C10.2, D2.2, G1.I, X1.2
- new net N$7: C11.1, G1.D
- net +12V: no longer D3.A, X1.2
- net +5V: now also C12.2, G1.Q; no longer U1.VOUT
- net GND: now also C10.1, C11.2, C12.1, D2.1, G1.GND; no longer C1.1, U1.GND

Commit message: ..
Parts:
- removed R14, R17, R8, R9: 47k, Resistor_smaller_fliegl:R-EU_WCAP-CSGP_0402
- added D3, D4, D5, D7: 150353GS74500, Wurth_LEDs_WL-SMDC:WL-SMDC_3535_150353GS74500
- added R19, R20, R23, R24: 100Ohm, Wurth_Resistor_WRIS-KWKB:WRIS-KWKB_0612_561020132008
- C10: value 47uF -> 22µF
- C4, C7, C8, C9: value 100 nF -> 10 nF; device Wurth_Capacitors_WCAP-CSGP:WCAP-CSGP_0402_885012205086_50V(DC) -> Wurth_Capacitors_WCAP-CSGP:WCAP-CSGP_0805_H0.8_885012207092_50V(DC)_R
Connections:
- new net N$1: D5.-, R19.1
- new net N$8: D4.-, R23.2
- new net N$9: D7.-, R24.2
- net +12V: now also J6.2; no longer J7.1
- net GND: now also J6.1, J6.3, J7.1, J7.2, J7.5, R19.2, R20.2, R23.1, R24.1; no longer R14.1, R17.2, R8.2, R9.1
- net N$6: now also D3.-, R20.1; no longer J6.5
- net Q1: now also D4.+, J6.4; no longer J7.2, R14.2
- net Q2: now also D3.+, J6.5; no longer J7.3, R17.1
- net Q3: now also D7.+, J7.3; no longer J7.4, R9.2
- net Q4: now also D5.+, J7.4; no longer J7.5, R8.1
Other:
- moved on the sheet: C5, C6, C7, C8, D1, J1, J6, R10, R11, R12, R13, R15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

Commit message: almost done, only cosmetics to do .
Parts:
- removed R11: 1k2, Resistor_smaller_fliegl:R-EU_WCAP-CSGP_0402
- removed R12, R15, R16, R5, R6: 4k7, Resistor_smaller_fliegl:R-EU_WCAP-CSGP_0402
- removed R21, R22: 60.4R 1%, Resistor_smaller_fliegl:R-0402_60.4OHMS_1%_AEC-Q200
- added J4, J8: (no value), Wurth_Connectors_WR-PHD:6130XX21121_61300621121
- C15: value 47 nF -> 47 nF; device fliegl-wuerth:WCAP-CSGP_0402_885012205054_25V(DC) -> Wurth_Capacitors_WCAP-CSGP:WCAP-CSGP_0805_H0.8_885012207096_50V(DC)_R
- C17, C19: value 100 nF -> 100 nF; device fliegl-wuerth:WCAP-CSGP_0402_885012205037_16V(DC) -> Wurth_Capacitors_WCAP-CSGP:WCAP-CSGP_0805_H0.8_885012207098_50V(DC)_R
- C2, C3, C5, C6: device Wurth_Capacitors_WCAP-CSGP:WCAP-CSGP_0402_885012205086_50V(DC) -> Wurth_Capacitors_WCAP-CSGP:WCAP-CSGP_0805_H0.8_885012207098_50V(DC)_R
- D2: value 26V -> 33V; device Wurth_EMC Components_WE-TVSP:WE-TVSP_DO-214AC_400W_BI_824501261 -> Wurth_EMC Components_WE-TVSP:WE-TVSP_DO-214AB_3000W_BI_824551331
- R1: value 1k2 -> 60R; device Resistor_smaller_fliegl:R-EU_WCAP-CSGP_0402 -> resistor:R-EU_R0805
- R10, R13, R18, R2, R4, R7: device Resistor_smaller_fliegl:R-EU_WCAP-CSGP_0402 -> resistor:R-EU_R0805
- R3: value 4k7 -> 60R; device Resistor_smaller_fliegl:R-EU_WCAP-CSGP_0402 -> resistor:R-EU_R0805
Connections:
- removed net +12V: C2.1, C3.1, C5.1, C6.1, D1.2, J6.2, U2.VS, U3.VS
- removed net +12V1: C10.2, D2.2, G1.I, X1.2
- removed net CAN_H: D6.2, R22.2, U4.CANH, X1.3
- removed net CAN_L: D6.1, R21.1, U4.CANL, X1.4
- removed net DENU2: R16.1
- removed net DENU3: R6.1
- removed net DSELU2: R12.1
- removed net DSELU3: R3.1
- removed net ISOU2: R11.2, R15.2, U2.IS
- removed net ISOU3: R1.2, R5.2, U3.IS
- removed net ISU2: R15.1
- removed net ISU3: R5.1
- removed net N$13: R12.2, U2.DSEL
- removed net N$15: R16.2, U2.DEN
- removed net N$3: R3.2, U3.DSEL
- removed net N$5: R6.2, U3.DEN
- new net CAN_N: D6.1, R3.2, U4.CANL, X1.4
- new net CAN_P: D6.2, R1.2, U4.CANH, X1.3
- new net ECU_PWR: C10.2, D2.2, G1.I, J8.2, J8.4, J8.6, X1.2
- new net PWR: C2.1, C3.1, C5.1, C6.1, D1.2, J6.2, J8.1, J8.3, J8.5, U2.VS, U3.VS
- new net PWR_GND: C4.1, C7.1, C8.2, C9.2, D1.1, J4.1, J4.3, J4.5, J6.1, J6.3, J7.1, J7.2, J7.5, R19.2, R20.2, R23.1, R24.1
- net GND: now also J4.2, J4.4, J4.6; no longer C4.1, C7.1, C8.2, C9.2, D1.1, J6.1, J6.3, J7.1, J7.2, J7.5, R1.1, R11.1, R19.2, R20.2, R23.1, R24.1
- net N$17: now also R1.1, R3.1; no longer R21.2, R22.1
Other:
- moved on the sheet: C15, C17, C19

Commit message: ok so far ..
Parts:
- removed D7: 150353GS74500, Wurth_LEDs_WL-SMDC:WL-SMDC_3535_150353GS74500
- added D0: 33V, Wurth_EMC Components_WE-TVSP:WE-TVSP_DO-214AB_3000W_BI_824551331
- D1, D2: value 33V -> 150353GS74500; device Wurth_EMC Components_WE-TVSP:WE-TVSP_DO-214AB_3000W_BI_824551331 -> Wurth_LEDs_WL-SMDC:WL-SMDC_3535_150353GS74500
- D5: value 150353GS74500 -> 33V; device Wurth_LEDs_WL-SMDC:WL-SMDC_3535_150353GS74500 -> Wurth_EMC Components_WE-TVSP:WE-TVSP_DO-214AB_3000W_BI_824551331
Connections:
- removed net GND: C10.1, C11.2, C12.1, C15.2, C17.2, C19.2, C2.2, C5.2, D2.1, D6.3, G1.GND, J2.1, J4.2, J4.4, J4.6, R10.1, R7.1, U4.GND, U4.NEN, X1.1
- new net ECU_GND: C10.1, C11.2, C12.1, C15.2, C17.2, C19.2, C2.2, C5.2, D5.1, D6.3, G1.GND, J2.1, J4.2, J4.4, J4.6, R10.1, R7.1, U4.GND, U4.NEN, X1.1
- net ECU_PWR: now also D5.2; no longer D2.2
- net N$1: now also D4.-; no longer D5.-
- net N$6: now also D2.-; no longer D3.-
- net N$8: now also D1.-; no longer D4.-
- net N$9: now also D3.-; no longer D7.-
- net PWR: now also D0.2; no longer D1.2
- net PWR_GND: now also D0.1; no longer D1.1
- net Q1: now also D1.+; no longer D4.+
- net Q2: now also D2.+; no longer D3.+
- net Q3: now also D3.+; no longer D7.+
- net Q4: now also D4.+; no longer D5.+
Other:
- note added: "https://obstwein-technik.eu/Core?aktiveNavigationsID=879&fachbetraegeID=209"
