File: Rail/pcb1.sch (EAGLE design)
At the start: 45 parts, among them J6 638207222005, J7 638207222005, U4 TLE9250VSJ, X1 S4P-VH

Commit message: nicer LED
Parts:
- D1, D2, D3, D4: value (none) -> 150141VS73100; device Wurth_LEDs_WL-SMRW:WL-SMRW_1206_DOME_156120VS82500_NOR -> Wurth_LEDs_WL-SMTW:WL-SMTW_3528_150141VS73100
- RX1, RX2, RX3, RX4: value 510mOhm -> 470Ohm; device Wurth_Resistor_WRIS-KWKH:WRIS-KWKH_0612_561070332078 -> Wurth_Resistor_WRIS-KWKB:WRIS-KWKB_0612_561020132023
Changed lines of the file:
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@@
 <part name="C12" library="Wurth_Capacitors_WCAP-CSGP" library_urn="urn:adsk.eagle:library:18488985" deviceset="WCAP-CSGP_0805_H1.25" device="_10V(DC)" package3d_urn="urn:adsk.eagle:package:18489127/2" technology="_885012107011" value="22  µF "/>
 <part name="D0" library="Wurth_EMC Components_WE-TVSP" library_urn="urn:adsk.eagle:library:14283044" deviceset="WE-TVSP_DO-214AB_3000W_BI" device="" package3d_urn="urn:adsk.eagle:package:12146529/2" technology="_824551331" value="33V"/>
-<part name="RX4" library="Wurth_Resistor_WRIS-KWKH" library_urn="urn:adsk.eagle:library:13353576" deviceset="WRIS-KWKH_0612" device="" package3d_urn="urn:adsk.eagle:package:13353581/2" technology="_561070332078" value="510mOhm"/>
-<part name="RX2" library="Wurth_Resistor_WRIS-KWKH" library_urn="urn:adsk.eagle:library:13353576" deviceset="WRIS-KWKH_0612" device="" package3d_urn="urn:adsk.eagle:package:13353581/2" technology="_561070332078" value="510mOhm"/>
-<part name="RX1" library="Wurth_Resistor_WRIS-KWKH" library_urn="urn:adsk.eagle:library:13353576" deviceset="WRIS-KWKH_0612" device="" package3d_urn="urn:adsk.eagle:package:13353581/2" technology="_561070332078" value="510mOhm"/>
-<part name="RX3" library="Wurth_Resistor_WRIS-KWKH" library_urn="urn:adsk.eagle:library:13353576" deviceset="WRIS-KWKH_0612" device="" package3d_urn="urn:adsk.eagle:package:13353581/2" technology="_561070332078" value="510mOhm"/>
+<part name="RX4" library="Wurth_Resistor_WRIS-KWKB" library_urn="urn:adsk.eagle:library:13351500" deviceset="WRIS-KWKB_0612" device="" package3d_urn="urn:adsk.eagle:package:13351506/2" technology="_561020132023" value="470Ohm"/>
+<part name="RX2" library="Wurth_Resistor_WRIS-KWKB" library_urn="urn:adsk.eagle:library:13351500" deviceset="WRIS-KWKB_0612" device="" package3d_urn="urn:adsk.eagle:package:13351506/2" technology="_561020132023" value="470Ohm"/>
+<part name="RX1" library="Wurth_Resistor_WRIS-KWKB" library_urn="urn:adsk.eagle:library:13351500" deviceset="WRIS-KWKB_0612" device="" package3d_urn="urn:adsk.eagle:package:13351506/2" technology="_561020132023" value="470Ohm"/>
+<part name="RX3" library="Wurth_Resistor_WRIS-KWKB" library_urn="urn:adsk.eagle:library:13351500" deviceset="WRIS-KWKB_0612" device="" package3d_urn="urn:adsk.eagle:package:13351506/2" technology="_561020132023" value="470Ohm"/>
 <part name="D5" library="Wurth_EMC Components_WE-TVSP" library_urn="urn:adsk.eagle:library:14283044" deviceset="WE-TVSP_DO-214AB_3000W_BI" device="" package3d_urn="urn:adsk.eagle:package:12146529/2" technology="_824551331" value="33V"/>
 <part name="R1" library="resistor" library_urn="urn:adsk.eagle:library:348" deviceset="R-EU_" device="R0805" package3d_urn="urn:adsk.eagle:package:23553/2" value="60R"/>
@@
 <part name="P+3" library="supply1" deviceset="+5V" device=""/>
 <part name="+3V3" library="supply1" deviceset="+3V3" device=""/>
-<part name="D2" library="Wurth_LEDs_WL-SMRW" library_urn="urn:adsk.eagle:library:19040144" deviceset="WL-SMRW_1206_DOME" device="_NOR" package3d_urn="urn:adsk.eagle:package:19040155/2" technology="_156120VS82500"/>
-<part name="D1" library="Wurth_LEDs_WL-SMRW" library_urn="urn:adsk.eagle:library:19040144" deviceset="WL-SMRW_1206_DOME" device="_NOR" package3d_urn="urn:adsk.eagle:package:19040155/2" technology="_156120VS82500"/>
-<part name="D4" library="Wurth_LEDs_WL-SMRW" library_urn="urn:adsk.eagle:library:19040144" deviceset="WL-SMRW_1206_DOME" device="_NOR" package3d_urn="urn:adsk.eagle:package:19040155/2" technology="_156120VS82500"/>
-<part name="D3" library="Wurth_LEDs_WL-SMRW" library_urn="urn:adsk.eagle:library:19040144" deviceset="WL-SMRW_1206_DOME" device="_NOR" package3d_urn="urn:adsk.eagle:package:19040155/2" technology="_156120VS82500"/>
+<part name="D2" library="Wurth_LEDs_WL-SMTW" library_urn="urn:adsk.eagle:library:19062651" deviceset="WL-SMTW_3528" device="" package3d_urn="urn:adsk.eagle:package:19062500/5" technology="_150141VS73100" value="150141VS73100"/>
+<part name="D1" library="Wurth_LEDs_WL-SMTW" library_urn="urn:adsk.eagle:library:19062651" deviceset="WL-SMTW_3528" device="" package3d_urn="urn:adsk.eagle:package:19062500/5" technology="_150141VS73100" value="150141VS73100"/>
+<part name="D4" library="Wurth_LEDs_WL-SMTW" library_urn="urn:adsk.eagle:library:19062651" deviceset="WL-SMTW_3528" device="" package3d_urn="urn:adsk.eagle:package:19062500/5" technology="_150141VS73100" value="150141VS73100"/>
+<part name="D3" library="Wurth_LEDs_WL-SMTW" library_urn="urn:adsk.eagle:library:19062651" deviceset="WL-SMTW_3528" device="" package3d_urn="urn:adsk.eagle:package:19062500/5" technology="_150141VS73100" value="150141VS73100"/>
 </parts>
 <sheets>
