File: Rail/pcb1_12V_XL.brd (EAGLE design)
At the start: 96.3 x 101.8 mm, 114 parts, among them J1 638207222006, J10 638207222006, J11 638207222006, J12 638207222006, J2 638207222006, U1 ESP32-S3-DEVKITC-1-N8R2, U4 TLE9250VSJ, X2 B4P-VH

Commit message: Prepare Prouction
Parts:
- removed C11: 100nF, Wurth_Capacitors_WCAP-CSGP:WCAP-CSGP_0402
- added J4: 61300421121, Wurth_Connectors_WR-PHD:61300421121
- G1: value TLE4270-2D-INF-PG-TO252-5-11_L_1 -> (none); device INF-PG-TO252-5-11L:INF-PG-TO252-5-11_L_1PRIMARY -> IFX27001TF V50:INF-PG-TO252-3-11_N
- moved G1 1.81 mm to (81.3, 64.8), turned to 135 degrees
- moved C12 1.38 mm to (81.1, 72.9), turned to 270 degrees
Connections:
- net N$16 renamed +6V
- removed net N$7: C11.1, G1.4
- net +5V: now also G1.2, J4.1, J4.2, J4.3, J4.4; no longer G1.5
- net ECU_GND: now also G1.1; no longer C11.2, G1.3
- net ECU_PWR: now also G1.3; no longer G1.1
Routing:
- net N$7: track 2.94 -> 0.00 mm
- net +5V: track 85.4 -> 82.6 mm, vias 3 -> 41
- net ECU_GND: vias 101 -> 78
- added copper zone on layer 1, net +5V
- added copper zone on layer 15, net +5V
- added copper zone on layer 16, net +5V
Other:
- board text added: "+5V"

Commit message: verpolschutz.
Parts:
- added C23: 330 µF, Wurth_Capacitors_WCAP-ASLI:WCAP-ASLI_12.5X14(DXL)
- added D006: MBRS340T3, fliegl-elektronik:SMC
- moved D5 3.81 mm to (88.6, 85.7)
Connections:
- new net N$3: C10.2, C23.1, D006.C, G1.3
- net ECU_GND: now also C23.2
- net ECU_PWR: now also D006.A; no longer C10.2, G1.3
Routing:
- net ECU_GND: vias 78 -> 76
- added copper zone on layer 1, net N$3
Changed lines of the file:
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@@
 <layer number="14" name="Route14" color="22" fill="1" visible="no" active="no"/>
 <layer number="15" name="Route15" color="23" fill="1" visible="no" active="yes"/>
-<layer number="16" name="Bottom" color="1" fill="1" visible="yes" active="yes"/>
-<layer number="17" name="Pads" color="2" fill="1" visible="no" active="yes"/>
+<layer number="16" name="Bottom" color="1" fill="1" visible="no" active="yes"/>
+<layer number="17" name="Pads" color="2" fill="1" visible="yes" active="yes"/>
 <layer number="18" name="Vias" color="2" fill="1" visible="yes" active="yes"/>
-<layer number="19" name="Unrouted" color="6" fill="1" visible="yes" active="yes"/>
+<layer number="19" name="Unrouted" color="6" fill="1" visible="no" active="yes"/>
 <layer number="20" name="Dimension" color="24" fill="1" visible="no" active="yes"/>
-<layer number="21" name="tPlace" color="7" fill="1" visible="no" active="yes"/>
+<layer number="21" name="tPlace" color="7" fill="1" visible="yes" active="yes"/>
 <layer number="22" name="bPlace" color="7" fill="1" visible="no" active="yes"/>
 <layer number="23" name="tOrigins" color="15" fill="1" visible="yes" active="yes"/>
@@
 <attribute name="NAME" x="34.798" y="18.23" size="0.8128" layer="25" align="bottom-center"/>
 </element>
-<element name="D5" library="Wurth_EMC Components_WE-TVSP" library_urn="urn:adsk.eagle:library:14283044" package="WE-TVSP_DO-214AB_BIDIRECTIONAL" package3d_urn="urn:adsk.eagle:package:12146529/2" value="33V" x="88.646" y="81.935" smashed="yes" rot="R180">
-<attribute name="DATASHEET-URL" value="https://www.we-online.com/catalog/datasheet/824551331.pdf" x="101.346" y="69.235" size="1.778" layer="27" rot="R180" display="off"/>
-<attribute name="IPEAK" value="56.3A" x="101.346" y="69.235" size="1.778" layer="27" rot="R180" display="off"/>
-<attribute name="MOUNT" value="SMT" x="101.346" y="69.235" size="1.778" layer="27" rot="R180" display="off"/>
-<attribute name="NAME" x="87.376" y="76.905" size="1.27" layer="25" rot="R180" align="bottom-center"/>
-<attribute name="PART-NUMBER" value=" 824551331 " x="101.346" y="69.235" size="1.778" layer="27" rot="R180" display="off"/>
-<attribute name="PDISS" value="3000W" x="101.346" y="69.235" size="1.778" layer="27" rot="R180" display="off"/>
-<attribute name="VALUE" x="91.896" y="86.775" size="1.27" layer="27" rot="R180"/>
-<attribute name="VBR" value="38.65V" x="101.346" y="69.235" size="1.778" layer="27" rot="R180" display="off"/>
-<attribute name="VCLAMP" value="53.3V" x="101.346" y="69.235" size="1.778" layer="27" rot="R180" display="off"/>
+<element name="D5" library="Wurth_EMC Components_WE-TVSP" library_urn="urn:adsk.eagle:library:14283044" package="WE-TVSP_DO-214AB_BIDIRECTIONAL" package3d_urn="urn:adsk.eagle:package:12146529/2" value="33V" x="88.646" y="85.745" smashed="yes" rot="R180">
+<attribute name="DATASHEET-URL" value="https://www.we-online.com/catalog/datasheet/824551331.pdf" x="101.346" y="73.045" size="1.778" layer="27" rot="R180" display="off"/>
+<attribute name="IPEAK" value="56.3A" x="101.346" y="73.045" size="1.778" layer="27" rot="R180" display="off"/>
+<attribute name="MOUNT" value="SMT" x="101.346" y="73.045" size="1.778" layer="27" rot="R180" display="off"/>
+<attribute name="NAME" x="87.376" y="80.715" size="1.27" layer="25" rot="R180" align="bottom-center"/>
+<attribute name="PART-NUMBER" value=" 824551331 " x="101.346" y="73.045" size="1.778" layer="27" rot="R180" display="off"/>
+<attribute name="PDISS" value="3000W" x="101.346" y="73.045" size="1.778" layer="27" rot="R180" display="off"/>
+<attribute name="VALUE" x="91.896" y="90.585" size="1.27" layer="27" rot="R180"/>
+<attribute name="VBR" value="38.65V" x="101.346" y="73.045" size="1.778" layer="27" rot="R180" display="off"/>
+<attribute name="VCLAMP" value="53.3V" x="101.346" y="73.045" size="1.778" layer="27" rot="R180" display="off"/>
 </element>
 <element name="R1" library="resistor" library_urn="urn:adsk.eagle:library:348" package="R0805" package3d_urn="urn:adsk.eagle:package:23553/2" value="60R" x="80.8388" y="82.53" smashed="yes" rot="R90">
@@
 <attribute name="VALUE" x="68.8924" y="58.2458" size="0.8128" layer="27" align="bottom-right"/>
 </element>
+<element name="D006" library="fliegl-elektronik" package="SMC" value="MBRS340T3" x="86.36" y="76.2" smashed="yes" rot="R90">
+<attribute name="ARTIKEL_NR" value="513891" x="85.09" y="76.2" size="1.778" layer="27" rot="R90" display="off"/>
+<attribute name="NAME" x="83.001" y="72.741" size="1.27" layer="25" rot="R90"/>
+<attribute name="VALUE" x="90.989" y="72.741" size="1.27" layer="27" rot="R90"/>
+</element>
+<element name="C23" library="Wurth_Capacitors_WCAP-ASLI" library_urn="urn:adsk.eagle:library:18353966" package="WCAP-ASLI_12.5X14(DXL)" package3d_urn="urn:adsk.eagle:package:18353982/3" value="330  µF " x="85.09" y="50.8" smashed="yes" rot="R180">
+<attribute name="DATASHEET-URL" value="https://www.we-online.com/catalog/datasheet/865080662019.pdf" x="85.09" y="50.8" size="1.778" layer="27" rot="R180" display="off"/>
+<attribute name="DF" value="12%" x="85.09" y="50.8" size="1.778" layer="27" rot="R180" display="off"/>
+<attribute name="DIAMETER" value="12.5mm" x="85.09" y="50.8" size="1.778" layer="27" rot="R180" display="off"/>
+<attribute name="I-LEAK" value="165uA" x="85.09" y="50.8" size="1.778" layer="27" rot="R180" display="off"/>
+<attribute name="I-RIPPLE" value="800mA" x="85.09" y="50.8" size="1.778" layer="27" rot="R180" display="off"/>
+<attribute name="L" value="14mm" x="85.09" y="50.8" size="1.778" layer="27" rot="R180" display="off"/>
+<attribute name="NAME" x="86.09" y="43" size="1.27" layer="25" rot="R180" align="bottom-center"/>
+<attribute name="OPERATING-TEMPERATURE" value="-55 °C up to +105 °C" x="85.09" y="50.8" size="1.778" layer="27" rot="R180" display="off"/>
+<attribute name="PART-NUMBER" value=" 865080662019 " x="85.09" y="50.8" size="1.778" layer="27" rot="R180" display="off"/>
+<attribute name="TECHNICAL-REFERENCE" value="ASEH140331M050DVCTGB000" x="85.09" y="50.8" size="1.778" layer="27" rot="R180" display="off"/>
+<attribute name="VALUE" x="85.79" y="59.7" size="1.27" layer="27" rot="R180" align="bottom-center"/>
+<attribute name="VR" value="50V(DC)" x="85.09" y="50.8" size="1.778" layer="27" rot="R180" display="off"/>
+</element>
 </elements>
 <signals>
@@
 </signal>
 <signal name="ECU_PWR">
-<contactref element="C10" pad="2"/>
-<polygon width="0.2032" layer="1" isolate="0.254">
-<vertex x="83.6812" y="40.8632"/>
+<polygon width="0.2032" layer="1" isolate="0.3048">
+<vertex x="83.6812" y="78.079653125"/>
 <vertex x="83.6812" y="97.19"/>
 <vertex x="89.47" y="97.19"/>
-<vertex x="89.47" y="40.8632"/>
+<vertex x="89.47" y="78.079653125"/>
 </polygon>
 <contactref element="D5" pad="2"/>
@@
 <wire x1="20.32" y1="96.52" x2="20.32" y2="91.44" width="1.27" layer="1"/>
 <wire x1="15.24" y1="96.52" x2="15.24" y2="91.44" width="1.27" layer="1"/>
-<contactref element="G1" pad="3"/>
+<contactref element="D006" pad="A"/>
 </signal>
 <signal name="N$1" class="1">
@@
 <via x="91.44" y="58.44" extent="1-16" drill="0.35"/>
 <via x="86.36" y="74.95" extent="1-16" drill="0.35"/>
-<via x="86.36" y="72.41" extent="1-16" drill="0.35"/>
-<via x="86.36" y="69.87" extent="1-16" drill="0.35"/>
 <via x="91.44" y="55.9" extent="1-16" drill="0.35"/>
 <via x="91.44" y="48.28" extent="1-16" drill="0.35"/>
@@
 <via x="81.28" y="58.44" extent="1-16" drill="0.35"/>
 <via x="81.28" y="59.71" extent="1-16" drill="0.35"/>
+<contactref element="C23" pad="2"/>
 </signal>
 <signal name="IX00">
@@
 <wire x1="87.63" y1="33.04" x2="87.63" y2="32.085" width="0.254" layer="1"/>
 </signal>
+<signal name="N$3">
+<contactref element="C10" pad="2"/>
+<contactref element="G1" pad="3"/>
+<contactref element="D006" pad="C"/>
+<contactref element="C23" pad="1"/>
+<polygon width="0.2032" layer="1" isolate="0.254" thermals="no">
+<vertex x="89.47" y="48.26"/>
+<vertex x="76.2" y="48.26"/>
+<vertex x="76.2" y="53.34"/>
+<vertex x="83.6812" y="53.34"/>
+<vertex x="83.6812" y="74.33"/>
+<vertex x="89.47" y="74.33"/>
+</polygon>
+</signal>
 </signals>
