File: Rail/pcb1_12V_XL.brd (EAGLE design)
At the start: 96.3 x 101.8 mm, 116 parts, among them J1 638207222006, J10 638207222006, J11 638207222006, J12 638207222006, J2 638207222006, J4 61300421121, U1 ESP32-S3-DEVKITC-1-N8R2, U4 TLE9250VSJ, X2 B4P-VH

Commit message: intermediate commit
Parts:
- moved R21 0.23 mm to (23.9, 85.7)
- moved R24 0.23 mm to (32.0, 85.7)
- moved R27 0.23 mm to (62.5, 85.7)
- moved R28 0.23 mm to (54.4, 85.7)
- moved R39 0.23 mm to (34.1, 85.7)
- moved R42 0.23 mm to (42.1, 85.7)
- moved R51 0.23 mm to (44.2, 85.7)
- moved R54 0.23 mm to (52.3, 85.7)
- moved C25 0.10 mm to (57.3, 85.7)
- moved C39 0.10 mm to (36.9, 85.7)
- moved C33 0.10 mm to (29.1, 85.7)
- moved C24 0.10 mm to (59.6, 85.7)
- moved C31 0.10 mm to (26.8, 85.7)
- moved C41 0.10 mm to (39.3, 85.7)
- moved C47 0.10 mm to (47.1, 85.7)
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Routing:
- net CAN_P: track 56.0 -> 58.4 mm
- net CI7: track 23.6 -> 24.7 mm
- net CI1: track 23.6 -> 24.5 mm
- net CI5: track 23.6 -> 24.4 mm
- net Q7C: track 37.9 -> 37.1 mm
- net AGNDU3: track 20.7 -> 20.0 mm
- net AGNDU5: track 20.7 -> 20.0 mm
- net CI6: track 26.0 -> 26.6 mm
- net CI2: track 26.0 -> 26.5 mm
- net ECU_GND: vias 76 -> 92

Commit message: generate 3D Model.
Parts:
- removed J10, J11, J12, J2: 638207222006, Wurth_Connectors_WR-FAST:638207222006
- added J13, J7: 638207222005, Wurth_Connectors_WR-FAST:638207222005
- added J15: 638207222008, Wurth_Connectors_WR-FAST:638207222008
- added J3, J6: 61302211821, Wurth_Connectors_WR-PHD:61302211821
- added J8: 638207222007, Wurth_Connectors_WR-FAST:638207222007
- J1: value 638207222006 -> 638207222005; device Wurth_Connectors_WR-FAST:638207222006 -> Wurth_Connectors_WR-FAST:638207222005
- moved J1 92.5 mm to (81.3, 7.62)
Connections:
- new net N$16: J7.2, J7.A2
- new net N$20: J13.5, J13.A5
- new net N$7: J7.4, J7.A4
- net ECU_GND: now also J7.1, J7.A1; no longer J2.5, J2.6, J2.A5, J2.A6
- net ECU_PWR: now also J7.3, J7.A3; no longer J2.3, J2.4, J2.A3, J2.A4
- net I1: now also J7.5, J7.A5; no longer J2.2, J2.A2
- net I2: now also J8.1, J8.A1; no longer J2.1, J2.A1
- net I3: now also J8.2, J8.A2; no longer J1.6, J1.A6
- net I4: now also J8.3, J8.A3; no longer J1.5, J1.A5
- net I5: now also J8.4, J8.A4; no longer J1.4, J1.A4
- net I6: now also J8.5, J8.A5; no longer J1.3, J1.A3
- net I7: now also J8.6, J8.A6; no longer J1.2, J1.A2
- net I8: now also J8.7, J8.A7; no longer J1.1, J1.A1
- net PWR: now also J13.4, J13.A4; no longer J10.2, J10.A2
- net PWR_GND: now also J1.1, J1.4, J1.5, J1.A1, J1.A4, J1.A5, J13.3, J13.A3, J15.3, J15.4, J15.7, J15.8, J15.A3, J15.A4, J15.A7, J15.A8; no longer J10.1, J10.3, J10.6, J10.A1, J10.A3, J10.A6, J11.1, J11.4, J11.5, J11.A1, J11.A4, J11.A5, J12.2, J12.3, J12.6, J12.A2, J12.A3, J12.A6
- net Q1: now also J13.2, J13.A2; no longer J10.4, J10.A4
- net Q2: now also J13.1, J13.A1; no longer J10.5, J10.A5
- net Q3: now also J15.6, J15.A6; no longer J11.2, J11.A2
- net Q4: now also J15.5, J15.A5; no longer J11.3, J11.A3
- net Q5: now also J15.2, J15.A2; no longer J11.6, J11.A6
- net Q6: now also J15.1, J15.A1; no longer J12.1, J12.A1
- net Q7: now also J1.3, J1.A3; no longer J12.4, J12.A4
- net Q8: now also J1.2, J1.A2; no longer J12.5, J12.A5
Routing:
- net N$7: track 0.00 -> 5.08 mm
- net ECU_PWR: track 10.2 -> 5.08 mm

Commit message: Connector 645004114822
Parts:
- removed X2: B4P-VH, con-JST VH:B4P-VH
- added J2: 645004114822, Wurth_Connectors_WR-WTB:645004114822
Connections:
- net CAN_N: now also J2.1; no longer X2.4
- net CAN_P: now also J2.2; no longer X2.3
- net ECU_GND: now also J2.4; no longer X2.1
- net ECU_PWR: now also J2.3; no longer X2.2
Changed lines of the file:
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@@
 <drawing>
 <settings>
-<setting alwaysvectorfont="yes"/>
+<setting alwaysvectorfont="no"/>
 <setting verticaltext="up"/>
 </settings>
-<grid distance="1.27" unitdist="mm" unit="mil" style="lines" multiple="1" display="yes" altdistance="10" altunitdist="mil" altunit="mm"/>
+<grid distance="10.62992" unitdist="mil" unit="mil" style="lines" multiple="1" display="yes" altdistance="10" altunitdist="mil" altunit="mm"/>
 <layers>
 <layer number="1" name="Top" color="4" fill="1" visible="yes" active="yes"/>
@@
 </layers>
 <board>
-<fusionsync huburn="a.YnVzaW5lc3M6bXNtdWM" projecturn="a.YnVzaW5lc3M6bXNtdWMjMjAyMjAzMTc1MDgxMzE4ODE" f3durn="urn:adsk.wipprod:dm.lineage:AZr2ohsdTDeaNf8dmFIMlA" pcbguid="" lastpulledtime="" lastsyncedchangeguid="" latestrevisionid="33f80b2f-3025-41da-9222-1f657163f287" lastsyncedrevisionid="33f80b2f-3025-41da-9222-1f657163f287" lastboardhashguid="8938bf13-636a-4ef8-5333-37305fbbb8bd" lastpushedtime="2023-08-04T22:23:09Z" linktopcb3d="false"/>
+<fusionsync huburn="a.YnVzaW5lc3M6bXNtdWM" projecturn="a.YnVzaW5lc3M6bXNtdWMjMjAyMjAzMTc1MDgxMzE4ODE" f3durn="urn:adsk.wipprod:dm.lineage:AZr2ohsdTDeaNf8dmFIMlA" pcbguid="" lastpulledtime="" lastsyncedchangeguid="" latestrevisionid="42242b72-a9b3-4739-a844-9cee953d63f4" lastsyncedrevisionid="42242b72-a9b3-4739-a844-9cee953d63f4" lastboardhashguid="9c99f7cd-cfef-2415-b362-01d43430a85c" lastpushedtime="2023-10-16T11:14:31Z" linktopcb3d="true"/>
 <plain>
 <wire x1="52.04" y1="41.46" x2="50.54" y2="41.46" width="0.1524" layer="22"/>
@@
 <attribute name="VALUE" x="-0.36" y="71.37" size="1.27" layer="27" rot="R270" align="top-left"/>
 </element>
-<element name="X2" library="con-JST VH" package="B4P-VH" value="B4P-VH" x="85.09" y="93.98" smashed="yes" rot="R180">
-<attribute name="NAME" x="93.57" y="94.615" size="1.27" layer="25" rot="R270" align="bottom-center"/>
-<attribute name="VALUE" x="91.03" y="97.155" size="1.27" layer="27" rot="R180"/>
-</element>
 <element name="U5" library="BTS7030-2EPA" package="SOP65P600X115-15N-V" value="" x="63.5" y="29.23" smashed="yes" rot="R270">
 <attribute name="NAME" x="66.77" y="28.474" size="0.8128" layer="25" font="vector" ratio="13" rot="SR0"/>
@@
 <attribute name="WORKING-VOLTAGE" value="300V(AC)" x="81.28" y="7.62" size="1.778" layer="27" rot="R180" display="off"/>
 </element>
+<element name="J2" library="Wurth_Connectors_WR-WTB" library_urn="urn:adsk.eagle:library:15818693" package="645004114822" package3d_urn="urn:adsk.eagle:package:15819025/2" value="645004114822" x="85.09" y="94.48" smashed="yes" rot="R180">
+<attribute name="CONTACT-RESISTANCE" value="20mOhm" x="85.09" y="94.48" size="1.778" layer="27" rot="R180" display="off"/>
+<attribute name="DATASHEET-URL" value="https://www.we-online.com/redexpert/spec/645004114822?ae" x="85.09" y="94.48" size="1.778" layer="27" rot="R180" display="off"/>
+<attribute name="GENDER" value="Male" x="85.09" y="94.48" size="1.778" layer="27" rot="R180" display="off"/>
+<attribute name="IR" value="7A" x="85.09" y="94.48" size="1.778" layer="27" rot="R180" display="off"/>
+<attribute name="L" value="15.84mm" x="85.09" y="94.48" size="1.778" layer="27" rot="R180" display="off"/>
+<attribute name="MOUNT" value="THT" x="85.09" y="94.48" size="1.778" layer="27" rot="R180" display="off"/>
+<attribute name="NAME" x="76.115" y="90.8" size="1.016" layer="25" rot="R180"/>
+<attribute name="PACKAGING" value="Bag" x="85.09" y="94.48" size="1.778" layer="27" rot="R180" display="off"/>
+<attribute name="PART-NUMBER" value="645004114822" x="85.09" y="94.48" size="1.778" layer="27" rot="R180" display="off"/>
+<attribute name="PCB-CABLE-PANEL" value="PCB" x="85.09" y="94.48" size="1.778" layer="27" rot="R180" display="off"/>
+<attribute name="PINS" value=" 4 " x="85.09" y="94.48" size="1.778" layer="27" rot="R180" display="off"/>
+<attribute name="PITCH" value="3.96mm" x="85.09" y="94.48" size="1.778" layer="27" rot="R180" display="off"/>
+<attribute name="TYPE" value="Vertical" x="85.09" y="94.48" size="1.778" layer="27" rot="R180" display="off"/>
+<attribute name="VALUE" x="76.09" y="93.58" size="1.016" layer="27" rot="R180"/>
+<attribute name="WORKING-VOLTAGE" value="250V(AC)" x="85.09" y="94.48" size="1.778" layer="27" rot="R180" display="off"/>
+</element>
 </elements>
 <signals>
@@
 <contactref element="U4" pad="7"/>
 <contactref element="R1" pad="2"/>
-<contactref element="X2" pad="3"/>
 <contactref element="D11" pad="2"/>
 <wire x1="53.975" y1="56.31" x2="53.975" y2="57.553" width="0.254" layer="1"/>
@@
 <wire x1="79.83453125" y1="76.2" x2="80.01" y2="76.2" width="0.254" layer="1"/>
 <wire x1="74.839" y1="74.126225" x2="76.912775" y2="76.2" width="0.254" layer="1"/>
+<contactref element="J2" pad="2"/>
 </signal>
 <signal name="CAN_N">
 <contactref element="U4" pad="6"/>
 <contactref element="R3" pad="2"/>
-<contactref element="X2" pad="4"/>
 <contactref element="D11" pad="1"/>
 <wire x1="52.705" y1="56.31" x2="52.705" y2="57.553" width="0.254" layer="1"/>
@@
 <wire x1="76.20000625" y1="76.20000625" x2="76.20000625" y2="77.46999375" width="0.254" layer="1"/>
 <wire x1="76.20000625" y1="77.46999375" x2="76.2" y2="77.47" width="0.254" layer="1"/>
+<contactref element="J2" pad="1"/>
 </signal>
 <signal name="+3V3">
@@
 <contactref element="J5" pad="4"/>
 <contactref element="J5" pad="6"/>
-<contactref element="X2" pad="2"/>
 <polygon width="0.2032" layer="1" isolate="0.254">
 <vertex x="82.4112" y="40.8632"/>
@@
 <contactref element="J7" pad="A3"/>
 <contactref element="J7" pad="3"/>
+<contactref element="J2" pad="3"/>
+<wire x1="85.146" y1="85.745" x2="87.07" y2="93.98" width="0" layer="19" extent="1-1"/>
+<wire x1="86.614" y1="41.93" x2="86.36" y2="79.9" width="0" layer="19" extent="1-1"/>
 </signal>
 <signal name="N$1" class="1">
@@
 <via x="81.661" y="76.855" extent="1-16" drill="0.35"/>
 <contactref element="D11" pad="3"/>
-<contactref element="X2" pad="1"/>
 <contactref element="G1" pad="1"/>
 <via x="80.01" y="58.44" extent="1-16" drill="0.35"/>
@@
 <contactref element="J7" pad="1"/>
 <contactref element="J7" pad="A1"/>
+<contactref element="J2" pad="4"/>
 <wire x1="63.5" y1="43.2" x2="62.23" y2="46.99" width="0" layer="19" extent="1-1"/>
 <wire x1="8.89" y1="46.99" x2="5.08" y2="50.82" width="0" layer="19" extent="1-1"/>
