File: Rail/pcb1_12V_XL.sch (EAGLE design)
At the start: 116 parts, among them J1 638207222006, J10 638207222006, J11 638207222006, J12 638207222006, J2 638207222006, J4 61300421121, U1 ESP32-S3-DEVKITC-1-N8R2, U4 TLE9250VSJ, X2 B4P-VH

Commit message: generate 3D Model.
Parts:
- removed J10, J11, J12, J2: 638207222006, Wurth_Connectors_WR-FAST:638207222006
- added J13, J7: 638207222005, Wurth_Connectors_WR-FAST:638207222005
- added J15: 638207222008, Wurth_Connectors_WR-FAST:638207222008
- added J3, J6: 61302211821, Wurth_Connectors_WR-PHD:6130XX11821_61302211821
- added J8: 638207222007, Wurth_Connectors_WR-FAST:638207222007
- J1: value 638207222006 -> 638207222005; device Wurth_Connectors_WR-FAST:638207222006 -> Wurth_Connectors_WR-FAST:638207222005
Connections:
- new net N$16: J7.2
- new net N$20: J13.5
- new net N$7: J7.4
- net ECU_GND: now also J7.1; no longer J2.5, J2.6
- net ECU_PWR: now also J7.3; no longer J2.3, J2.4
- net I1: now also J7.5; no longer J2.2
- net I2: now also J8.1; no longer J2.1
- net I3: now also J8.2; no longer J1.6
- net I4: now also J8.3; no longer J1.5
- net I5: now also J8.4; no longer J1.4
- net I6: now also J8.5; no longer J1.3
- net I7: now also J8.6; no longer J1.2
- net I8: now also J8.7; no longer J1.1
- net PWR: now also J13.4; no longer J10.2
- net PWR_GND: now also J1.1, J1.4, J1.5, J13.3, J15.3, J15.4, J15.7, J15.8; no longer J10.1, J10.3, J10.6, J11.1, J11.4, J11.5, J12.2, J12.3, J12.6
- net Q1: now also J13.2; no longer J10.4
- net Q2: now also J13.1; no longer J10.5
- net Q3: now also J15.6; no longer J11.2
- net Q4: now also J15.5; no longer J11.3
- net Q5: now also J15.2; no longer J11.6
- net Q6: now also J15.1; no longer J12.1
- net Q7: now also J1.3; no longer J12.4
- net Q8: now also J1.2; no longer J12.5

Commit message: Connector 645004114822
Parts:
- removed X2: B4P-VH, con-JST VH:B4P-VH
- added J2: 645004114822, Wurth_Connectors_WR-WTB:645004114822
Connections:
- net CAN_N: now also J2.1; no longer X2.4
- net CAN_P: now also J2.2; no longer X2.3
- net ECU_GND: now also J2.4; no longer X2.1
- net ECU_PWR: now also J2.3; no longer X2.2
Changed lines of the file:
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@@
 <part name="PWR_GND19" library="supply_isobus" deviceset="PWR_GND" device=""/>
 <part name="PWR_GND20" library="supply_isobus" deviceset="PWR_GND" device=""/>
-<part name="X2" library="con-JST VH" deviceset="B4P-VH" device=""/>
 <part name="U5" library="BTS7030-2EPA" deviceset="BTS7030-2EPA" device=""/>
 <part name="R5" library="resistor" library_urn="urn:adsk.eagle:library:348" deviceset="R-EU_" device="R0805" package3d_urn="urn:adsk.eagle:package:23553/2" value="4k7"/>
@@
 <part name="J15" library="Wurth_Connectors_WR-FAST" library_urn="urn:adsk.eagle:library:15267884" deviceset="638207222008" device="" package3d_urn="urn:adsk.eagle:package:15267957/3" value=" 638207222008 "/>
 <part name="J1" library="Wurth_Connectors_WR-FAST" library_urn="urn:adsk.eagle:library:15267884" deviceset="638207222005" device="" package3d_urn="urn:adsk.eagle:package:15267960/3" value=" 638207222005 "/>
+<part name="J2" library="Wurth_Connectors_WR-WTB" library_urn="urn:adsk.eagle:library:15818693" deviceset="645004114822" device="" package3d_urn="urn:adsk.eagle:package:15819025/2" value="645004114822"/>
 </parts>
 <sheets>
@@
 <attribute name="VALUE" x="-22.86" y="48.26" size="1.778" layer="96"/>
 </instance>
-<instance part="X2" gate="G$1" x="-30.48" y="137.16" smashed="yes" rot="MR270">
-<attribute name="VALUE" x="-20.32" y="138.43" size="1.778" layer="96" rot="MR270"/>
-<attribute name="NAME" x="-36.322" y="138.43" size="1.778" layer="95" rot="MR270"/>
-</instance>
 <instance part="ECU_GND28" gate="ECU_GND" x="-25.4" y="119.38" smashed="yes">
 <attribute name="VALUE" x="-27.94" y="116.84" size="1.778" layer="96"/>
@@
 <attribute name="NAME" x="11.86" y="67.215" size="1.4224" layer="95" rot="R90" align="bottom-center"/>
 <attribute name="VALUE" x="20.315" y="66.955" size="1.4224" layer="96" rot="R90" align="bottom-center"/>
+</instance>
+<instance part="J2" gate="G$1" x="-27.94" y="149.86" smashed="yes" rot="MR0">
+<attribute name="NAME" x="-35.58" y="148.205" size="1.016" layer="95" rot="MR0"/>
+<attribute name="VALUE" x="-35.32" y="146.8" size="1.016" layer="96" rot="MR0"/>
 </instance>
 </instances>
@@
 <net name="CAN_P" class="0">
 <segment>
-<wire x1="-30.48" y1="129.54" x2="-30.48" y2="119.38" width="0.1524" layer="91"/>
+<wire x1="-30.48" y1="144.78" x2="-30.48" y2="119.38" width="0.1524" layer="91"/>
 <wire x1="-30.48" y1="119.38" x2="-43.18" y2="119.38" width="0.1524" layer="91"/>
 <label x="-43.18" y="119.38" size="1.778" layer="95" rot="R180" xref="yes"/>
-<pinref part="X2" gate="G$1" pin="3"/>
+<pinref part="J2" gate="G$1" pin="2"/>
+<junction x="-30.48" y="144.78"/>
+<wire x1="-30.48" y1="144.78" x2="-30.48" y2="129.54" width="0.1524" layer="91"/>
 </segment>
 </net>
 <net name="CAN_N" class="0">
 <segment>
-<wire x1="-33.02" y1="129.54" x2="-33.02" y2="127" width="0.1524" layer="91"/>
+<wire x1="-33.02" y1="144.78" x2="-33.02" y2="127" width="0.1524" layer="91"/>
 <wire x1="-33.02" y1="127" x2="-43.18" y2="127" width="0.1524" layer="91"/>
 <label x="-43.18" y="127" size="1.778" layer="95" rot="R180" xref="yes"/>
-<pinref part="X2" gate="G$1" pin="4"/>
+<pinref part="J2" gate="G$1" pin="1"/>
+<junction x="-33.02" y="144.78"/>
+<wire x1="-33.02" y1="144.78" x2="-33.02" y2="129.54" width="0.1524" layer="91"/>
 </segment>
 </net>
@@
 </segment>
 <segment>
-<wire x1="-27.94" y1="129.54" x2="-27.94" y2="127" width="0.1524" layer="91"/>
+<wire x1="-27.94" y1="144.78" x2="-27.94" y2="127" width="0.1524" layer="91"/>
 <pinref part="ECU_PWR3" gate="ECU_PWR" pin="ECU_PWR"/>
 <wire x1="-12.7" y1="127" x2="-27.94" y2="127" width="0.1524" layer="91"/>
-<pinref part="X2" gate="G$1" pin="2"/>
+<pinref part="J2" gate="G$1" pin="3"/>
+<junction x="-27.94" y="144.78"/>
+<wire x1="-27.94" y1="144.78" x2="-27.94" y2="129.54" width="0.1524" layer="91"/>
 </segment>
 </net>
@@
 </segment>
 <segment>
-<pinref part="X2" gate="G$1" pin="1"/>
 <pinref part="ECU_GND28" gate="ECU_GND" pin="ECU_GND"/>
-<wire x1="-25.4" y1="129.54" x2="-25.4" y2="121.92" width="0.1524" layer="91"/>
-</segment>
-</net>
+<wire x1="-25.4" y1="144.78" x2="-25.4" y2="121.92" width="0.1524" layer="91"/>
+<pinref part="J2" gate="G$1" pin="4"/>
+<junction x="-25.4" y="144.78"/>
+<wire x1="-25.4" y1="144.78" x2="-25.4" y2="129.54" width="0.1524" layer="91"/>
+</segment>
+</net>
