File: C3_Stamp/M5_STACK_STAMP_C3_8P_6P.brd (EAGLE design)
At the start: 20.3 x 22.9 mm, 3 parts, among them J1 61300811121, J2 61300611121

Commit message: 8P 6P Header
Other:
- board size 20.3 x 22.9 mm -> 20.3 x 35.6 mm
Changed lines of the file:
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@@
 <drawing>
 <settings>
-<setting alwaysvectorfont="no"/>
+<setting alwaysvectorfont="yes"/>
 <setting verticaltext="up"/>
 </settings>
@@
 <board>
 <plain>
-<wire x1="0" y1="12.7" x2="20.3" y2="12.7" width="0" layer="20"/>
-<wire x1="20.3" y1="12.7" x2="20.32" y2="35.56" width="0" layer="20"/>
+<wire x1="0" y1="0" x2="20.3" y2="0" width="0" layer="20"/>
+<wire x1="20.3" y1="0" x2="20.32" y2="35.56" width="0" layer="20"/>
 <wire x1="20.32" y1="35.56" x2="0" y2="35.56" width="0" layer="20"/>
-<wire x1="0" y1="35.56" x2="0" y2="12.7" width="0" layer="20"/>
+<wire x1="0" y1="35.56" x2="0" y2="0" width="0" layer="20"/>
 </plain>
 <attributes>
