File: S3/ISOBUS_Hardware_S3.sch (EAGLE design)
At the start: 13 parts, among them IC1 MCP2562-E_P, J1 61304421821, J2 61304421821, J3 DTF13-4P

Commit message: Order
Parts:
- added D1: 1N4004, Diodes:1N4004
- added D2: 15KEXXC, diode:15KEXXC
Connections:
- new net RST: J1.39, J1.40
- net +12V: now also D1.C; no longer J3.1
- net G4: now also J1.37, J1.38; no longer J1.39, J1.40
- net G5: now also J1.35, J1.36; no longer J1.37, J1.38
- net GND: now also D2.1
- net N$2: now also D1.A, D2.2, J3.1; no longer J1.35, J1.36

Commit message: Done !
Connections:
- net CAN_N renamed CAN_L
- net CAN_P renamed CAN_H
