File: S3/ISOBUS_Hardware_S3.brd (EAGLE design)
At the start: 76.2 x 55.9 mm, 13 parts, among them IC1 MCP2562-E_P, J1 61304421821, J2 61304421821, J3 DTF13-4P

Commit message: Order
Parts:
- added D1: 1N4004, Diodes:DO-41
- added D2: 15KEXXC, diode:CB429-17
- moved J3 10.2 mm to (54.6, 10.2)
Connections:
- new net RST: J1.39, J1.40
- net +12V: now also D1.C; no longer J3.1
- net G4: now also J1.37, J1.38; no longer J1.39, J1.40
- net G5: now also J1.35, J1.36; no longer J1.37, J1.38
- net GND: now also D2.A
- net N$2: now also D1.A, D2.C, J3.1; no longer J1.35, J1.36
Routing:
- net N$2: track 2.54 -> 31.3 mm
- net +12V: track 26.3 -> 18.6 mm
- net +5V: track 76.6 -> 83.7 mm
- net CAN_N: track 22.0 -> 27.6 mm
- net GND: track 2.54 -> 0.00 mm, vias 13 -> 16
- net RST: track 0.00 -> 2.54 mm
- net CAN_P: track 29.6 -> 31.1 mm
- net G4: track 42.3 -> 41.3 mm
Other:
- board text added: "ANT"
- board text added: "USB here"

Commit message: Done !
Connections:
- net CAN_N renamed CAN_L
- net CAN_P renamed CAN_H
Changed lines of the file:
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@@
 <wire x1="48.995" y1="25.42" x2="49.015" y2="25.4" width="1.27" layer="1"/>
 </signal>
-<signal name="CAN_P">
+<signal name="CAN_H">
 <contactref element="J3" pad="2"/>
 <contactref element="IC1" pad="7"/>
@@
 <wire x1="57.501975" y1="6.701975" x2="59.06" y2="8.26" width="0.508" layer="1"/>
 </signal>
-<signal name="CAN_N">
+<signal name="CAN_L">
 <contactref element="J3" pad="4"/>
 <contactref element="IC1" pad="6"/>

Commit message: ..
Changed lines of the file:
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@@
 </layers>
 <board>
+<fusionsync huburn="a.YnVzaW5lc3M6bXNtdWM" projecturn="a.YnVzaW5lc3M6bXNtdWMjRDIwMjAwMTIwMjU2OTQxODgx" f3durn="urn:adsk.wipprod:dm.lineage:ExIlnZevT6uYyBvQXCN5Vw" pcbguid="" lastpulledtime="2022-02-26T11:21:51Z" lastsyncedchangeguid="" latestrevisionid="20f162bb-cff4-4575-98db-a538cf2787c5" lastsyncedrevisionid="20f162bb-cff4-4575-98db-a538cf2787c5" lastboardhashguid="ddf9a8c5-966c-32ee-8878-5549e6081f18" lastpushedtime="2022-02-26T11:19:37Z" linktopcb3d="true"/>
 <plain>
+<text x="19.05" y="-22.86" size="1.778" layer="21">USB here</text>
+<text x="-3.81" y="-22.86" size="1.778" layer="21">USB here</text>
+<text x="1.27" y="29.21" size="1.778" layer="21">ANT</text>
+<hole x="56.835" y="-4.815" drill="3"/>
+<hole x="56.835" y="16.015" drill="3"/>
+<wire x1="-13.97" y1="31.75" x2="-13.97" y2="-24.13" width="0" layer="20"/>
 <wire x1="-13.97" y1="-24.13" x2="62.21" y2="-24.13" width="0" layer="20"/>
 <wire x1="62.21" y1="-24.13" x2="62.23" y2="31.75" width="0" layer="20"/>
 <wire x1="62.23" y1="31.75" x2="-13.97" y2="31.75" width="0" layer="20"/>
-<wire x1="-13.97" y1="31.75" x2="-13.97" y2="-24.13" width="0" layer="20"/>
-<text x="19.05" y="-22.86" size="1.778" layer="21">USB here</text>
-<text x="-3.81" y="-22.86" size="1.778" layer="21">USB here</text>
-<text x="1.27" y="29.21" size="1.778" layer="21">ANT</text>
 </plain>
 <attributes>
@@
 <via x="7.62" y="8.89" extent="1-16" drill="1.1"/>
 <via x="19.05" y="15.24" extent="1-16" drill="1.1"/>
+<wire x1="35.56" y1="27.94" x2="41.91" y2="27.92" width="0" layer="19" extent="1-1"/>
+<wire x1="27.94" y1="25.4" x2="35.56" y2="27.94" width="0" layer="19" extent="1-1"/>
+<wire x1="20.32" y1="27.94" x2="27.94" y2="25.4" width="0" layer="19" extent="1-1"/>
+<wire x1="15.24" y1="30.48" x2="20.32" y2="27.94" width="0" layer="19" extent="1-1"/>
+<wire x1="12.7" y1="30.48" x2="15.24" y2="30.48" width="0" layer="19" extent="1-1"/>
+<wire x1="8.89" y1="24.13" x2="12.7" y2="30.48" width="0" layer="19" extent="1-1"/>
+<wire x1="2.54" y1="22.86" x2="8.89" y2="24.13" width="0" layer="19" extent="1-1"/>
+<wire x1="-1.27" y1="27.94" x2="2.54" y2="22.86" width="0" layer="19" extent="1-1"/>
+<wire x1="7.62" y1="17.78" x2="8.89" y2="24.13" width="0" layer="19" extent="1-1"/>
+<wire x1="2.54" y1="13.97" x2="7.62" y2="17.78" width="0" layer="19" extent="1-1"/>
+<wire x1="-3.81" y1="20.32" x2="2.54" y2="22.86" width="0" layer="19" extent="1-1"/>
+<wire x1="0" y1="7.62" x2="2.54" y2="13.97" width="0" layer="19" extent="1-1"/>
+<wire x1="7.62" y1="8.89" x2="2.54" y2="13.97" width="0" layer="19" extent="1-1"/>
+<wire x1="33.02" y1="15.24" x2="27.94" y2="25.4" width="0" layer="19" extent="1-1"/>
+<wire x1="38.1" y1="15.24" x2="33.02" y2="15.24" width="0" layer="19" extent="1-1"/>
+<wire x1="25.4" y1="12.7" x2="33.02" y2="15.24" width="0" layer="19" extent="1-1"/>
+<wire x1="22.86" y1="12.7" x2="25.4" y2="12.7" width="0" layer="19" extent="1-1"/>
+<wire x1="19.05" y1="15.24" x2="22.86" y2="12.7" width="0" layer="19" extent="1-1"/>
+<wire x1="19.05" y1="8.89" x2="22.86" y2="12.7" width="0" layer="19" extent="1-1"/>
+<wire x1="19.05" y1="3.81" x2="19.05" y2="8.89" width="0" layer="19" extent="1-1"/>
+<wire x1="30.48" y1="5.08" x2="25.4" y2="12.7" width="0" layer="19" extent="1-1"/>
+<wire x1="38.1" y1="2.54" x2="30.48" y2="5.08" width="0" layer="19" extent="1-1"/>
+<wire x1="45.72" y1="0" x2="38.1" y2="2.54" width="0" layer="19" extent="1-1"/>
+<wire x1="26.67" y1="-6.35" x2="30.48" y2="5.08" width="0" layer="19" extent="1-1"/>
+<wire x1="2.54" y1="-5.08" x2="0" y2="7.62" width="0" layer="19" extent="1-1"/>
+<wire x1="7.62" y1="-10.16" x2="2.54" y2="-5.08" width="0" layer="19" extent="1-1"/>
+<wire x1="12.7" y1="-20.32" x2="7.62" y2="-10.16" width="0" layer="19" extent="1-1"/>
+<wire x1="12.7" y1="-22.86" x2="12.7" y2="-20.32" width="0" layer="19" extent="1-1"/>
+<wire x1="15.24" y1="-22.86" x2="12.7" y2="-22.86" width="0" layer="19" extent="1-1"/>
+<wire x1="15.24" y1="-20.32" x2="12.7" y2="-20.32" width="0" layer="19" extent="1-1"/>
+<wire x1="59.06" y1="1.04" x2="45.72" y2="0" width="0" layer="19" extent="1-1"/>
+<wire x1="-6.35" y1="-15.24" x2="2.54" y2="-5.08" width="0" layer="19" extent="1-1"/>
+<wire x1="-10.16" y1="-22.86" x2="-6.35" y2="-15.24" width="0" layer="19" extent="1-1"/>
+<wire x1="-12.7" y1="-22.86" x2="-10.16" y2="-22.86" width="0" layer="19" extent="1-1"/>
 </signal>
 <signal name="+12V">
@@
 </note>
 <note version="8.3" severity="warning">
+Since Version 8.3, EAGLE supports Fusion synchronisation.
+This feature will not be available in this version and saving
+the document will break the link to the Fusion PCB feature.
+</note>
+<note version="8.3" severity="warning">
