File: ButtonBoards/6ButtonTHT/6ButtonTHT.brd (EAGLE design)
At the start: 48.3 x 66 mm, 22 parts, among them J1 4P-2.0-90D

Commit message: pdf
Parts:
- removed J2: (no value), jumper:JUMP
- removed JP1: (no value), jumper:JP2
Connections:
- removed net C: C3.2, JP1.2, R11.2, R7.1, R8.2
- net A: no longer JP1.3
- net B: now also C3.2, R11.2, R7.1, R8.2; no longer JP1.1
Routing:
- net C: track 26.4 -> 0.00 mm
- net A: track 6.88 -> 0.00 mm
- net B: track 10.3 -> 13.4 mm
Changed lines of the file:
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@@
 <attribute name="VALUE" x="35.2806" y="-45.085" size="1.27" layer="27" ratio="10" rot="R180"/>
-</element>
-<element name="JP1" library="jumper" library_urn="urn:adsk.eagle:library:252" package="JP2" package3d_urn="urn:adsk.eagle:package:15452/1" value="" x="35.56" y="-58.42" smashed="yes" rot="R270">
-<attribute name="NAME" x="37.211" y="-54.864" size="1.27" layer="25" ratio="10" rot="R270"/>
-<attribute name="POPULARITY" value="34" x="35.56" y="-58.42" size="1.778" layer="27" rot="R270" display="off"/>
-<attribute name="VALUE" x="31.242" y="-54.864" size="1.27" layer="27" ratio="10" rot="R270"/>
-</element>
-<element name="J2" library="jumper" library_urn="urn:adsk.eagle:library:252" package="JUMP" package3d_urn="urn:adsk.eagle:package:15453/1" value="" x="40.64" y="-59.69" smashed="yes" rot="R180">
-<attribute name="NAME" x="40.84" y="-60.29" size="0.1" layer="25" rot="R180"/>
-<attribute name="POPULARITY" value="0" x="40.64" y="-59.69" size="1.778" layer="27" rot="R180" display="off"/>
-<attribute name="VALUE" x="40.94" y="-58.99" size="0.1" layer="27" rot="R180"/>
 </element>
 <element name="D1" library="diode" library_urn="urn:adsk.eagle:library:210" package="SOD81" package3d_urn="urn:adsk.eagle:package:43363/2" value="BZD23" x="17.78" y="-50.8" smashed="yes">
@@
 <signal name="B">
 <contactref element="J1" pad="2"/>
-<contactref element="JP1" pad="1"/>
 <wire x1="27.162" y1="-58.42" x2="27.94" y2="-55.88" width="1.016" layer="16"/>
-<wire x1="27.94" y1="-55.88" x2="35.56" y2="-55.88" width="1.016" layer="16"/>
+<contactref element="C3" pad="2"/>
+<contactref element="R8" pad="2"/>
+<contactref element="R7" pad="1"/>
+<contactref element="R11" pad="2"/>
+<wire x1="27.94" y1="-45.72" x2="25.4" y2="-45.72" width="1.016" layer="16"/>
+<wire x1="25.4" y1="-45.72" x2="25.4" y2="-48.26" width="1.016" layer="16"/>
+<wire x1="25.4" y1="-48.26" x2="30.48" y2="-50.8" width="1.016" layer="16"/>
+<wire x1="30.48" y1="-50.8" x2="27.94" y2="-55.88" width="0" layer="19" extent="16-16"/>
 </signal>
 <signal name="A">
 <contactref element="J1" pad="1"/>
-<contactref element="JP1" pad="3"/>
-<wire x1="29.162" y1="-58.42" x2="35.56" y2="-60.96" width="1.016" layer="16"/>
 </signal>
 <signal name="N$1">
@@
 <wire x1="38" y1="-40.6" x2="40.64" y2="-40.64" width="1.016" layer="16"/>
 </signal>
-<signal name="C">
-<contactref element="C3" pad="2"/>
-<contactref element="R8" pad="2"/>
-<contactref element="R7" pad="1"/>
-<contactref element="JP1" pad="2"/>
-<wire x1="38.1" y1="-58.42" x2="35.56" y2="-58.42" width="1.016" layer="16"/>
-<contactref element="R11" pad="2"/>
-<wire x1="27.94" y1="-45.72" x2="25.4" y2="-45.72" width="1.016" layer="16"/>
-<wire x1="25.4" y1="-45.72" x2="25.4" y2="-48.26" width="1.016" layer="16"/>
-<wire x1="25.4" y1="-48.26" x2="30.48" y2="-50.8" width="1.016" layer="16"/>
-<wire x1="30.48" y1="-50.8" x2="38.1" y2="-53.34" width="1.016" layer="16"/>
-<wire x1="38.1" y1="-53.34" x2="38.1" y2="-58.42" width="1.016" layer="16"/>
-</signal>
 <signal name="+3V3">

Commit message: THT
Connections:
- net A: now also C3.2, R11.2, R7.1, R8.2
- net B: no longer C3.2, R11.2, R7.1, R8.2
Routing:
- net A: track 0.00 -> 18.9 mm
- net B: track 13.4 -> 0.00 mm
- net GND: track 61.5 -> 64.0 mm
Other:
- outline, holes or cut-outs redrawn
Changed lines of the file:
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@@
 <setting verticaltext="up"/>
 </settings>
-<grid distance="100" unitdist="mil" unit="mil" style="lines" multiple="1" display="yes" altdistance="5" altunitdist="mil" altunit="mil"/>
+<grid distance="1" unitdist="mm" unit="mm" style="lines" multiple="1" display="yes" altdistance="5" altunitdist="mil" altunit="mil"/>
 <layers>
 <layer number="1" name="Top" color="4" fill="1" visible="yes" active="yes"/>
@@
 <layer number="43" name="vRestrict" color="2" fill="10" visible="yes" active="yes"/>
 <layer number="44" name="Drills" color="7" fill="1" visible="no" active="yes"/>
-<layer number="45" name="Holes" color="7" fill="1" visible="no" active="yes"/>
+<layer number="45" name="Holes" color="7" fill="1" visible="yes" active="yes"/>
 <layer number="46" name="Milling" color="3" fill="1" visible="no" active="yes"/>
 <layer number="47" name="Measures" color="7" fill="1" visible="no" active="yes"/>
@@
 <board>
 <plain>
-<wire x1="0" y1="0" x2="48.24" y2="0" width="0" layer="20"/>
-<wire x1="48.24" y1="0" x2="48.26" y2="-66.04" width="0" layer="20"/>
-<wire x1="48.26" y1="-66.04" x2="0" y2="-66.04" width="0" layer="20"/>
-<wire x1="0" y1="-66.04" x2="0" y2="0" width="0" layer="20"/>
+<wire x1="0" y1="-64.44" x2="0" y2="-1.6" width="0" layer="20"/>
+<wire x1="0" y1="-1.6" x2="1.6" y2="0" width="0" layer="20" curve="-90"/>
+<wire x1="1.6" y1="0" x2="46.640484375" y2="0" width="0" layer="20"/>
+<wire x1="46.640484375" y1="0" x2="48.240484375" y2="-1.59940625" width="0" layer="20" curve="-89.978738"/>
+<wire x1="48.240484375" y1="-1.59940625" x2="48.259515625" y2="-64.44059375" width="0" layer="20"/>
+<wire x1="48.259515625" y1="-64.44059375" x2="46.659515625" y2="-66.04" width="0" layer="20" curve="-90.017345"/>
+<wire x1="46.659515625" y1="-66.04" x2="1.6" y2="-66.04" width="0" layer="20"/>
+<wire x1="1.6" y1="-66.04" x2="0" y2="-64.44" width="0" layer="20" curve="-90"/>
+<hole x="3" y="-3" drill="3.2"/>
+<hole x="45" y="-3" drill="3.2"/>
+<hole x="45" y="-63" drill="3.2"/>
+<hole x="3" y="-63" drill="3.2"/>
 </plain>
 <attributes>
@@
 </element>
 <element name="R2" library="rcl" library_urn="urn:adsk.eagle:library:334" package="0207/10" package3d_urn="urn:adsk.eagle:package:23491/2" value="15K" x="40.64" y="-20.32" smashed="yes" rot="R270">
-<attribute name="NAME" x="44.704" y="-17.272" size="1.27" layer="25" ratio="10" rot="R270"/>
+<attribute name="NAME" x="42.704" y="-19.272" size="1.27" layer="25" ratio="10" rot="R270"/>
 <attribute name="POPULARITY" value="81" x="40.64" y="-20.32" size="1.778" layer="27" rot="R270" display="off"/>
 <attribute name="SPICEPREFIX" value="R" x="40.64" y="-20.32" size="1.778" layer="27" rot="R270" display="off"/>
-<attribute name="VALUE" x="40.005" y="-18.0594" size="1.27" layer="27" ratio="10" rot="R270"/>
+<attribute name="VALUE" x="40.005" y="-19.0594" size="1.27" layer="27" ratio="10" rot="R270"/>
 </element>
 <element name="R3" library="rcl" library_urn="urn:adsk.eagle:library:334" package="0207/10" package3d_urn="urn:adsk.eagle:package:23491/2" value="9.1K" x="7.62" y="-27.94" smashed="yes" rot="R270">
@@
 </element>
 <element name="R4" library="rcl" library_urn="urn:adsk.eagle:library:334" package="0207/10" package3d_urn="urn:adsk.eagle:package:23491/2" value="5.6K" x="40.64" y="-33.02" smashed="yes" rot="R270">
-<attribute name="NAME" x="44.704" y="-29.972" size="1.27" layer="25" ratio="10" rot="R270"/>
+<attribute name="NAME" x="42.704" y="-29.972" size="1.27" layer="25" ratio="10" rot="R270"/>
 <attribute name="POPULARITY" value="81" x="40.64" y="-33.02" size="1.778" layer="27" rot="R270" display="off"/>
 <attribute name="SPICEPREFIX" value="R" x="40.64" y="-33.02" size="1.778" layer="27" rot="R270" display="off"/>
@@
 <attribute name="MOUSER_PRICE-STOCK" value="https://www.mouser.com/Search/Refine.aspx?Keyword=810-FG28X7R1H473KNT6" x="19.05" y="-50.8" size="1.778" layer="27" display="off"/>
 <attribute name="NAME" x="25.4" y="-45.72" size="1.27" layer="25" align="center"/>
-<attribute name="VALUE" x="30.48" y="-45.72" size="1.27" layer="27" align="center"/>
+<attribute name="VALUE" x="37.72" y="-56.52" size="1.27" layer="27" rot="R90" align="center"/>
 </element>
 <element name="R7" library="rcl" library_urn="urn:adsk.eagle:library:334" package="0207/10" package3d_urn="urn:adsk.eagle:package:23491/2" value="10K" x="20.32" y="-48.26" smashed="yes" rot="R180">
@@
 <attribute name="POPULARITY" value="81" x="33.02" y="-45.72" size="1.778" layer="27" rot="R180" display="off"/>
 <attribute name="SPICEPREFIX" value="R" x="33.02" y="-45.72" size="1.778" layer="27" rot="R180" display="off"/>
-<attribute name="VALUE" x="35.2806" y="-45.085" size="1.27" layer="27" ratio="10" rot="R180"/>
+<attribute name="VALUE" x="33.2806" y="-48.085" size="1.27" layer="27" ratio="10" rot="R180"/>
 </element>
 <element name="D1" library="diode" library_urn="urn:adsk.eagle:library:210" package="SOD81" package3d_urn="urn:adsk.eagle:package:43363/2" value="BZD23" x="17.78" y="-50.8" smashed="yes">
@@
 <wire x1="22.86" y1="-55.88" x2="23.162" y2="-58.42" width="1.016" layer="16"/>
 <wire x1="22.86" y1="-50.8" x2="22.76" y2="-40.6" width="1.016" layer="16"/>
-<wire x1="22.86" y1="-50.8" x2="25.4" y2="-50.8" width="0" layer="19" extent="1-1"/>
+<wire x1="22.86" y1="-50.8" x2="25.4" y2="-50.8" width="1.016" layer="16"/>
 </signal>
 <signal name="+5V">
@@
 <signal name="B">
 <contactref element="J1" pad="2"/>
-<wire x1="27.162" y1="-58.42" x2="27.94" y2="-55.88" width="1.016" layer="16"/>
+</signal>
+<signal name="A">
+<contactref element="J1" pad="1"/>
 <contactref element="C3" pad="2"/>
 <contactref element="R8" pad="2"/>
@@
 <wire x1="25.4" y1="-45.72" x2="25.4" y2="-48.26" width="1.016" layer="16"/>
 <wire x1="25.4" y1="-48.26" x2="30.48" y2="-50.8" width="1.016" layer="16"/>
-<wire x1="30.48" y1="-50.8" x2="27.94" y2="-55.88" width="0" layer="19" extent="16-16"/>
-</signal>
-<signal name="A">
-<contactref element="J1" pad="1"/>
+<wire x1="30.48" y1="-50.8" x2="30.48" y2="-57.102" width="1.016" layer="16"/>
+<wire x1="30.48" y1="-57.102" x2="29.162" y2="-58.42" width="1.016" layer="16"/>
 </signal>
 <signal name="N$1">
@@
 <contactref element="S3" pad="4"/>
 <contactref element="R3" pad="1"/>
-<wire x1="7.62" y1="-22.86" x2="10.16" y2="-22.86" width="1.016" layer="16"/>
-<wire x1="10.16" y1="-22.86" x2="10.26" y2="-22.9" width="0" layer="19" extent="16-16"/>
+<wire x1="10.26" y1="-22.9" x2="10.22" y2="-22.86" width="1.016" layer="16"/>
+<wire x1="10.22" y1="-22.86" x2="7.62" y2="-22.86" width="1.016" layer="16"/>
 </signal>
 <signal name="N$4">
@@
 <wire x1="12.7" y1="-50.8" x2="15.24" y2="-53.34" width="1.016" layer="16"/>
 </signal>
-<signal name="N$9">
-<via x="2.54" y="-5.08" extent="1-16" drill="1"/>
-</signal>
-<signal name="N$10">
-<via x="5.08" y="-5.08" extent="1-16" drill="1"/>
-</signal>
 <signal name="N$11">
 <via x="7.62" y="-5.08" extent="1-16" drill="1"/>
@@
 <via x="40.64" y="-5.08" extent="1-16" drill="1"/>
 </signal>
-<signal name="N$25">
-<via x="43.18" y="-5.08" extent="1-16" drill="1"/>
-</signal>
-<signal name="N$26">
-<via x="45.72" y="-5.08" extent="1-16" drill="1"/>
-</signal>
 <signal name="N$27">
