File: ButtonBoards/6ButtonTHT/6ButtonTHT.sch (EAGLE design)
At the start: 22 parts, among them J1 4P-2.0-90D

Commit message: pdf
Parts:
- removed J2: (no value), jumper:JUMPER
- removed JP1: (no value), jumper:JP2E
Connections:
- removed net C: C3.2, JP1.2, R11.2, R7.1, R8.2
- net A: no longer JP1.3
- net B: now also C3.2, R11.2, R7.1, R8.2; no longer JP1.1
Other:
- moved on the sheet: C3, D1, J1, R1, R10, R11, R2, R3, R4, R5, R6, R7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

Commit message: THT
Connections:
- net A: now also C3.2, R11.2, R7.1, R8.2
- net B: no longer C3.2, R11.2, R7.1, R8.2
Changed lines of the file:
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@@
 <label x="287.02" y="66.04" size="1.27" layer="95" rot="R180" xref="yes"/>
+</segment>
+</net>
+<net name="A" class="0">
+<segment>
+<pinref part="J1" gate="G$1" pin="1"/>
+<wire x1="300.99" y1="68.58" x2="287.02" y2="68.58" width="0.1524" layer="91"/>
+<label x="287.02" y="68.58" size="1.27" layer="95" rot="R180" xref="yes"/>
 </segment>
 <segment>
@@
 </segment>
 </net>
-<net name="A" class="0">
-<segment>
-<pinref part="J1" gate="G$1" pin="1"/>
-<wire x1="300.99" y1="68.58" x2="287.02" y2="68.58" width="0.1524" layer="91"/>
-<label x="287.02" y="68.58" size="1.27" layer="95" rot="R180" xref="yes"/>
-</segment>
-</net>
