File: ButtonBoards/6ButtonSMD/6ButtonSMD.brd (EAGLE design)
At the start: 48.3 x 66 mm, 20 parts, among them J1 4P-2.0-90D

Commit message: SMD
Parts:
- C3: value FG28X7R1H473KNT06 -> 47nF; device FG28X7R1H473KNT06-pcb-part-libraries:FG28 -> Wurth_Capacitors_WCAP-CSGP:WCAP-CSGP_1206_H0.8
- D1: value BZD23 -> 3.3V; device diode:SOD81 -> diode:SOD80C
- J1: value 4P-2.0-90D -> 4P-SMD-2.0-90D; device OPL_Connector:HW4-2.0-90D -> OPL_Connector:HW4-SMD-2.0-90D
- R1, R10, R11, R2, R3, R4, R5, R6, R7, R8, R9: device rcl:0207/10 -> rcl:R1206
- S1, S2, S3, S4, S5, S6: value (none) -> 430162073826; device Wurth_Switch_WS-TATV:4304X60737X6 -> Wurth_Switch_WS-TASV:430162073826
- moved R5 3.59 mm to (5.08, -38.1)
- moved R1 2.84 mm to (5.08, -14.0)
- moved R3 2.84 mm to (5.08, -26.7)
- moved R2 2.84 mm to (43.2, -19.1)
- moved R10 2.54 mm to (17.8, -53.3)
- moved R11 2.54 mm to (17.8, -45.7)
- moved R4 2.54 mm to (43.2, -33.0)
- moved R6 2.54 mm to (43.2, -45.7)
- moved R7 2.54 mm to (17.8, -48.3)
- moved R9 2.54 mm to (17.8, -55.9)
- moved R8 1.80 mm to (34.3, -47.0)
- moved S2 1.27 mm to (33.0, -12.7)
- moved S4 1.27 mm to (33.0, -25.4)
- moved S6 1.27 mm to (33.0, -38.1)
- moved S1 1.27 mm to (15.2, -12.7)
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Routing:
- net GND: track 64.0 -> 0.00 mm
- net N$30: track 38.7 -> 0.00 mm
- net N$27: track 36.8 -> 0.00 mm
- net A: track 18.9 -> 0.00 mm
- net +3V3: track 9.72 -> 0.00 mm
- net +5V: track 5.09 -> 0.00 mm
- net N$3: track 2.66 -> 0.00 mm
- net N$6: track 2.64 -> 0.00 mm
- net N$4: track 2.64 -> 0.00 mm
- net N$2: track 2.64 -> 0.00 mm
- net N$5: track 2.64 -> 0.00 mm
- net N$1: track 2.64 -> 0.00 mm
