File: XL-accessories/Board_4_Buttons.brd (EAGLE design)
At the start: 156 x 47.9 mm, 0 parts

Commit message: ..
Parts:
- added J1: (no value), Wurth_Connectors_WR-TBL Rising Cage Clamp:691508110305
Connections:
- new net N$1: J1.1, J1.2, J1.3, J1.4, J1.5
Routing:
- net N$1: track 0.00 -> 14.1 mm
Other:
- outline, holes or cut-outs redrawn
