File: XL-accessories/Board_4_Poti.brd (EAGLE design)
At the start: 156 x 47.9 mm, 0 parts

Commit message: ..
Parts:
- added J1, J2: (no value), Wurth_Connectors_WR-TBL Rising Cage Clamp:691508110305
Connections:
- new net N$2: J1.1, J1.2, J1.3, J1.4, J1.5
- new net N$3: J2.1, J2.2, J2.3, J2.4, J2.5
Routing:
- net N$3: track 0.00 -> 14.0 mm
- net N$2: track 0.00 -> 14.0 mm
Changed lines of the file:
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@@
 </autorouter>
 <elements>
+<element name="J1" library="Wurth_Connectors_WR-TBL Rising Cage Clamp" library_urn="urn:adsk.eagle:library:16280519" package="691508110305" package3d_urn="urn:adsk.eagle:package:16248440/3" value="" x="-15" y="20" smashed="yes" rot="R180">
+<attribute name="DATASHEET-URL" value="https://www.we-online.com/catalog/datasheet/691508110305.pdf" x="-15" y="20" size="1.778" layer="27" font="vector" rot="R180" display="off"/>
+<attribute name="IR-UL" value="10A" x="-15" y="20" size="1.778" layer="27" font="vector" rot="R180" display="off"/>
+<attribute name="MOUNT" value="THT" x="-15" y="20" size="1.778" layer="27" font="vector" rot="R180" display="off"/>
+<attribute name="NAME" x="-15" y="12" size="1.27" layer="25" rot="R180" align="bottom-center"/>
+<attribute name="PART-NUMBER" value=" 691508110305 " x="-15" y="20" size="1.778" layer="27" font="vector" rot="R180" display="off"/>
+<attribute name="PINS" value=" 5 " x="-15" y="20" size="1.778" layer="27" font="vector" rot="R180" display="off"/>
+<attribute name="PITCH" value="3.5mm" x="-15" y="20" size="1.778" layer="27" font="vector" rot="R180" display="off"/>
+<attribute name="TYPE" value="Horizontal" x="-15" y="20" size="1.778" layer="27" font="vector" rot="R180" display="off"/>
+<attribute name="VALUE" x="-11.5" y="25.5" size="1.27" layer="27" rot="R180"/>
+<attribute name="WIRE" value="30 to 16 (AWG) 0.05 to 1.31 (mm²)" x="-15" y="20" size="1.778" layer="27" font="vector" rot="R180" display="off"/>
+<attribute name="WORKING-VOLTAGE-UL" value="300V (AC)" x="-15" y="20" size="1.778" layer="27" font="vector" rot="R180" display="off"/>
+</element>
+<element name="J2" library="Wurth_Connectors_WR-TBL Rising Cage Clamp" library_urn="urn:adsk.eagle:library:16280519" package="691508110305" package3d_urn="urn:adsk.eagle:package:16248440/3" value="" x="15" y="20" smashed="yes" rot="R180">
+<attribute name="DATASHEET-URL" value="https://www.we-online.com/catalog/datasheet/691508110305.pdf" x="15" y="20" size="1.778" layer="27" font="vector" rot="R180" display="off"/>
+<attribute name="IR-UL" value="10A" x="15" y="20" size="1.778" layer="27" font="vector" rot="R180" display="off"/>
+<attribute name="MOUNT" value="THT" x="15" y="20" size="1.778" layer="27" font="vector" rot="R180" display="off"/>
+<attribute name="NAME" x="15" y="12" size="1.27" layer="25" rot="R180" align="bottom-center"/>
+<attribute name="PART-NUMBER" value=" 691508110305 " x="15" y="20" size="1.778" layer="27" font="vector" rot="R180" display="off"/>
+<attribute name="PINS" value=" 5 " x="15" y="20" size="1.778" layer="27" font="vector" rot="R180" display="off"/>
+<attribute name="PITCH" value="3.5mm" x="15" y="20" size="1.778" layer="27" font="vector" rot="R180" display="off"/>
+<attribute name="TYPE" value="Horizontal" x="15" y="20" size="1.778" layer="27" font="vector" rot="R180" display="off"/>
+<attribute name="VALUE" x="18.5" y="25.5" size="1.27" layer="27" rot="R180"/>
+<attribute name="WIRE" value="30 to 16 (AWG) 0.05 to 1.31 (mm²)" x="15" y="20" size="1.778" layer="27" font="vector" rot="R180" display="off"/>
+<attribute name="WORKING-VOLTAGE-UL" value="300V (AC)" x="15" y="20" size="1.778" layer="27" font="vector" rot="R180" display="off"/>
+</element>
 </elements>
 <signals>
+<signal name="N$2">
+<contactref element="J1" pad="5"/>
+<contactref element="J1" pad="4"/>
+<contactref element="J1" pad="1"/>
+<contactref element="J1" pad="2"/>
+<contactref element="J1" pad="3"/>
+<wire x1="-22" y1="15.05" x2="-18.5" y2="15.05" width="2.54" layer="1"/>
+<wire x1="-8" y1="15.05" x2="-11.5" y2="15.05" width="2.54" layer="1"/>
+<wire x1="-15" y1="15.05" x2="-11.5" y2="15.05" width="2.54" layer="1"/>
+<wire x1="-18.5" y1="15.05" x2="-15" y2="15.05" width="2.54" layer="1"/>
+</signal>
+<signal name="N$3">
+<contactref element="J2" pad="1"/>
+<contactref element="J2" pad="5"/>
+<contactref element="J2" pad="2"/>
+<contactref element="J2" pad="3"/>
+<contactref element="J2" pad="4"/>
+<wire x1="8" y1="15.05" x2="11.5" y2="15.05" width="2.54" layer="1"/>
+<wire x1="22" y1="15.05" x2="18.5" y2="15.05" width="2.54" layer="1"/>
+<wire x1="15" y1="15.05" x2="18.5" y2="15.05" width="2.54" layer="1"/>
+<wire x1="11.5" y1="15.05" x2="15" y2="15.05" width="2.54" layer="1"/>
+</signal>
 </signals>
 <mfgpreviewcolors>
@@
 </board>
 </drawing>
+<compatibility>
+<note version="8.2" severity="warning">
+Since Version 8.2, EAGLE supports online libraries. The ids
+of those online libraries will not be understood (or retained)
+with this version.
+</note>
+<note version="8.3" severity="warning">
+Since Version 8.3, EAGLE supports URNs for individual library
+assets (packages, symbols, and devices). The URNs of those assets
+will not be understood (or retained) with this version.
+</note>
+<note version="8.3" severity="warning">
+Since Version 8.3, EAGLE supports the association of 3D packages
+with devices in libraries, schematics, and board files. Those 3D
+packages will not be understood (or retained) with this version.
+</note>
+</compatibility>
 </eagle>
