File: XL-accessories/Board_4_Wippen.brd (EAGLE design)
At the start: 156 x 47.9 mm, 0 parts

Commit message: ..
Parts:
- added J1: (no value), Wurth_Connectors_WR-TBL Rising Cage Clamp:691508110305
Connections:
- new net N$1: J1.1, J1.2, J1.3, J1.4, J1.5
Changed lines of the file:
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@@
 <layer number="48" name="Document" color="7" fill="1" visible="yes" active="yes"/>
 <layer number="49" name="Reference" color="7" fill="1" visible="yes" active="yes"/>
+<layer number="50" name="dxf" color="7" fill="1" visible="no" active="no"/>
 <layer number="51" name="tDocu" color="7" fill="1" visible="yes" active="yes"/>
 <layer number="52" name="bDocu" color="7" fill="1" visible="yes" active="yes"/>
+<layer number="88" name="SimResults" color="9" fill="1" visible="no" active="no"/>
+<layer number="89" name="SimProbes" color="9" fill="1" visible="no" active="no"/>
+<layer number="90" name="Modules" color="5" fill="1" visible="no" active="no"/>
+<layer number="91" name="Nets" color="2" fill="1" visible="no" active="no"/>
+<layer number="92" name="Busses" color="1" fill="1" visible="no" active="no"/>
+<layer number="93" name="Pins" color="2" fill="1" visible="no" active="no"/>
+<layer number="94" name="Symbols" color="4" fill="1" visible="no" active="no"/>
+<layer number="95" name="Names" color="7" fill="1" visible="no" active="no"/>
+<layer number="96" name="Values" color="7" fill="1" visible="no" active="no"/>
+<layer number="97" name="Info" color="7" fill="1" visible="no" active="no"/>
+<layer number="98" name="Guide" color="6" fill="1" visible="no" active="no"/>
+<layer number="250" name="Descript" color="7" fill="1" visible="yes" active="yes"/>
+<layer number="251" name="SMDround" color="7" fill="1" visible="yes" active="yes"/>
 </layers>
 <board>
@@
 </autorouter>
 <elements>
+<element name="J1" library="Wurth_Connectors_WR-TBL Rising Cage Clamp" library_urn="urn:adsk.eagle:library:16280519" package="691508110305" package3d_urn="urn:adsk.eagle:package:16248440/3" value="" x="0" y="20" smashed="yes" rot="R180">
+<attribute name="DATASHEET-URL" value="https://www.we-online.com/catalog/datasheet/691508110305.pdf" x="0" y="20" size="1.778" layer="27" font="vector" rot="R180" display="off"/>
+<attribute name="IR-UL" value="10A" x="0" y="20" size="1.778" layer="27" font="vector" rot="R180" display="off"/>
+<attribute name="MOUNT" value="THT" x="0" y="20" size="1.778" layer="27" font="vector" rot="R180" display="off"/>
+<attribute name="NAME" x="0" y="12" size="1.27" layer="25" rot="R180" align="bottom-center"/>
+<attribute name="PART-NUMBER" value=" 691508110305 " x="0" y="20" size="1.778" layer="27" font="vector" rot="R180" display="off"/>
+<attribute name="PINS" value=" 5 " x="0" y="20" size="1.778" layer="27" font="vector" rot="R180" display="off"/>
+<attribute name="PITCH" value="3.5mm" x="0" y="20" size="1.778" layer="27" font="vector" rot="R180" display="off"/>
+<attribute name="TYPE" value="Horizontal" x="0" y="20" size="1.778" layer="27" font="vector" rot="R180" display="off"/>
+<attribute name="VALUE" x="3.5" y="25.5" size="1.27" layer="27" rot="R180"/>
+<attribute name="WIRE" value="30 to 16 (AWG) 0.05 to 1.31 (mm²)" x="0" y="20" size="1.778" layer="27" font="vector" rot="R180" display="off"/>
+<attribute name="WORKING-VOLTAGE-UL" value="300V (AC)" x="0" y="20" size="1.778" layer="27" font="vector" rot="R180" display="off"/>
+</element>
 </elements>
 <signals>
+<signal name="N$1">
+<contactref element="J1" pad="1"/>
+<contactref element="J1" pad="2"/>
+<contactref element="J1" pad="5"/>
+<contactref element="J1" pad="3"/>
+<contactref element="J1" pad="4"/>
+<wire x1="3.5" y1="15.05" x2="7" y2="15.05" width="0" layer="19" extent="1-1"/>
+<wire x1="0" y1="15.05" x2="3.5" y2="15.05" width="0" layer="19" extent="1-1"/>
+<wire x1="-3.5" y1="15.05" x2="0" y2="15.05" width="0" layer="19" extent="1-1"/>
+<wire x1="-7" y1="15.05" x2="-3.5" y2="15.05" width="0" layer="19" extent="1-1"/>
+</signal>
 </signals>
 <mfgpreviewcolors>
@@
 </board>
 </drawing>
+<compatibility>
+<note version="8.2" severity="warning">
+Since Version 8.2, EAGLE supports online libraries. The ids
+of those online libraries will not be understood (or retained)
+with this version.
+</note>
+<note version="8.3" severity="warning">
+Since Version 8.3, EAGLE supports URNs for individual library
+assets (packages, symbols, and devices). The URNs of those assets
+will not be understood (or retained) with this version.
+</note>
+<note version="8.3" severity="warning">
+Since Version 8.3, EAGLE supports the association of 3D packages
+with devices in libraries, schematics, and board files. Those 3D
+packages will not be understood (or retained) with this version.
+</note>
+</compatibility>
 </eagle>
