File: Hutschienenmoped-XL_2ETH/Hutschienenmoped-XL_2ETH.brd (EAGLE design)
At the start: 166.3 x 101.8 mm, 129 parts, among them J1 638207222005, J13 638207222005, J15 638207222008, J2 645004114822, J4 61300421121, J7 638207222005, J8 638207222007, U4 TLE9250VSJ

Commit message: Update Fusion 360 sync details and add new signal connections. Add text labels for USB, PRG, and PSRAM on the schematic sheet.
Connections:
- new net N$16: ESP32-J3.15
- new net N$21: ESP32-J3.16
- new net N$22: ESP32-J1.20
- new net N$23: ESP32-J1.17
- new net N$24: ESP32-J1.16
- new net N$25: ESP32-J1.14
- new net N$26: ESP32-J1.12
- new net N$27: ESP32-J1.9
- new net N$7: ESP32-J3.10
Changed lines of the file:
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@@
 </layers>
 <board>
-<fusionsync huburn="a.YnVzaW5lc3M6bXNtdWM" projecturn="a.YnVzaW5lc3M6bXNtdWMjMjAyMjAzMTc1MDgxMzE4ODE" f3durn="urn:adsk.wipprod:dm.lineage:ajjTPt2gRBKkWSmyFLQsrw" pcbguid="" lastpulledtime="2023-10-23T01:33:52Z" lastsyncedchangeguid="" latestrevisionid="4beeb25c-c3ea-4695-891d-5bfc398b937a" lastsyncedrevisionid="4beeb25c-c3ea-4695-891d-5bfc398b937a" lastboardhashguid="d47e81b0-323d-8e0b-e760-b965a1c6aebf" lastpushedtime="2024-03-24T11:47:00Z" linktopcb3d="true"/>
+<fusionsync huburn="a.YnVzaW5lc3M6bXNtdWM" projecturn="a.YnVzaW5lc3M6bXNtdWMjMjAyMjAzMTc1MDgxMzE4ODE" f3durn="urn:adsk.wipprod:dm.lineage:ajjTPt2gRBKkWSmyFLQsrw" pcbguid="" lastpulledtime="2023-10-23T01:33:52Z" lastsyncedchangeguid="" latestrevisionid="868574ed-2542-4ae0-a29b-ef24def32971" lastsyncedrevisionid="868574ed-2542-4ae0-a29b-ef24def32971" lastboardhashguid="f227f1a2-26d9-5c76-6985-b8a639230d9e" lastpushedtime="2024-03-24T12:42:37Z" linktopcb3d="true"/>
 <plain>
 <wire x1="52.04" y1="41.46" x2="50.54" y2="41.46" width="0.1524" layer="22"/>
@@
 <contactref element="W1-J2" pad="3"/>
 </signal>
+<signal name="N$7">
+<contactref element="ESP32-J3" pad="10"/>
+</signal>
+<signal name="N$16">
+<contactref element="ESP32-J3" pad="15"/>
+</signal>
+<signal name="N$21">
+<contactref element="ESP32-J3" pad="16"/>
+</signal>
+<signal name="N$22">
+<contactref element="ESP32-J1" pad="20"/>
+</signal>
+<signal name="N$23">
+<contactref element="ESP32-J1" pad="17"/>
+</signal>
+<signal name="N$24">
+<contactref element="ESP32-J1" pad="16"/>
+</signal>
+<signal name="N$25">
+<contactref element="ESP32-J1" pad="14"/>
+</signal>
+<signal name="N$26">
+<contactref element="ESP32-J1" pad="12"/>
+</signal>
+<signal name="N$27">
+<contactref element="ESP32-J1" pad="9"/>
+</signal>
 </signals>
