File: XL-accessories/Board_4_Buttons/Board_4_Buttons_WS-TASV_ SMD Plug.brd (EAGLE design)
At the start: 156 x 47.9 mm, 5 parts, among them J2 691709710305

Commit message: Update package and device set information for WS-TASV SMD Plug.
Parts:
- S1, S2, S3, S4: value 430162073826 -> 430162043826; device Wurth_Switch_WS-TASV:430162073826 -> Wurth_Switch_WS-TASV:430162043826
Changed lines of the file:
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@@
 </layers>
 <board>
-<fusionsync huburn="a.YnVzaW5lc3M6bXNtdWM" projecturn="a.YnVzaW5lc3M6bXNtdWMjMjAyMjAzMTc1MDgxMzE4ODE" f3durn="urn:adsk.wipprod:dm.lineage:DrcSPxU1SBmPMhIK7kDvdw" pcbguid="9b75bbeb-fb64-421f-af9e-c77acb5c75e7" lastpulledtime="" lastsyncedchangeguid="" latestrevisionid="5f049106-6f64-49cb-ae9b-23230f38e5ce" lastsyncedrevisionid="5f049106-6f64-49cb-ae9b-23230f38e5ce" lastboardhashguid="a641f209-cf45-be64-c272-31e8228ba700" lastpushedtime="2025-03-01T07:48:16Z" linktopcb3d="true"/>
+<fusionsync huburn="a.YnVzaW5lc3M6bXNtdWM" projecturn="a.YnVzaW5lc3M6bXNtdWMjMjAyMjAzMTc1MDgxMzE4ODE" f3durn="urn:adsk.wipprod:dm.lineage:DrcSPxU1SBmPMhIK7kDvdw" pcbguid="" lastpulledtime="" lastsyncedchangeguid="" latestrevisionid="5f049106-6f64-49cb-ae9b-23230f38e5ce" lastsyncedrevisionid="5f049106-6f64-49cb-ae9b-23230f38e5ce" lastboardhashguid="a641f209-cf45-be64-c272-31e8228ba700" lastpushedtime="2025-03-01T07:48:16Z" linktopcb3d="true"/>
 <plain>
 <wire x1="-60" y1="-20" x2="-73" y2="-20" width="0" layer="20"/>
@@
 </autorouter>
 <elements>
-<element name="S1" library="Wurth_Switch_WS-TASV" library_urn="urn:adsk.eagle:library:18304196" package="430162073826" package3d_urn="urn:adsk.eagle:package:18304357/2" value="430162073826" x="-45" y="0" smashed="yes">
-<attribute name="DATASHEET-URL" value="https://www.we-online.com/redexpert/spec/430162073826?ae" x="-45" y="0" size="1.778" layer="27" display="off"/>
-<attribute name="HEIGHT" value="7.3mm" x="-45" y="0" size="1.778" layer="27" display="off"/>
+<element name="S1" library="Wurth_Switch_WS-TASV" library_urn="urn:adsk.eagle:library:18304196" package="430162043826" package3d_urn="urn:adsk.eagle:package:18304303/2" value="430162043826" x="-45" y="0" smashed="yes">
+<attribute name="DATASHEET-URL" value="https://www.we-online.com/redexpert/spec/430162043826?ae" x="-45" y="0" size="1.778" layer="27" display="off"/>
+<attribute name="HEIGHT" value="4.3mm" x="-45" y="0" size="1.778" layer="27" display="off"/>
 <attribute name="NAME" x="-45.034" y="6.9177" size="1.27" layer="25" align="bottom-center"/>
 <attribute name="OPERATION-FORCE" value="260g" x="-45" y="0" size="1.778" layer="27" display="off"/>
-<attribute name="PART-NUMBER" value="430162073826" x="-45" y="0" size="1.778" layer="27" display="off"/>
-<attribute name="QTY" value=" 250 " x="-45" y="0" size="1.778" layer="27" display="off"/>
-<attribute name="VALUE" value="430162073826" x="-48.494" y="-7.8258" size="1.27" layer="27"/>
-</element>
-<element name="S2" library="Wurth_Switch_WS-TASV" library_urn="urn:adsk.eagle:library:18304196" package="430162073826" package3d_urn="urn:adsk.eagle:package:18304357/2" value="430162073826" x="-15" y="0" smashed="yes">
-<attribute name="DATASHEET-URL" value="https://www.we-online.com/redexpert/spec/430162073826?ae" x="-15" y="0" size="1.778" layer="27" display="off"/>
-<attribute name="HEIGHT" value="7.3mm" x="-15" y="0" size="1.778" layer="27" display="off"/>
+<attribute name="PART-NUMBER" value="430162043826" x="-45" y="0" size="1.778" layer="27" display="off"/>
+<attribute name="QTY" value=" 400 " x="-45" y="0" size="1.778" layer="27" display="off"/>
+<attribute name="VALUE" value="430162043826" x="-48.494" y="-7.8258" size="1.27" layer="27"/>
+</element>
+<element name="S2" library="Wurth_Switch_WS-TASV" library_urn="urn:adsk.eagle:library:18304196" package="430162043826" package3d_urn="urn:adsk.eagle:package:18304303/2" value="430162043826" x="-15" y="0" smashed="yes">
+<attribute name="DATASHEET-URL" value="https://www.we-online.com/redexpert/spec/430162043826?ae" x="-15" y="0" size="1.778" layer="27" display="off"/>
+<attribute name="HEIGHT" value="4.3mm" x="-15" y="0" size="1.778" layer="27" display="off"/>
 <attribute name="NAME" x="-15.034" y="6.9177" size="1.27" layer="25" align="bottom-center"/>
 <attribute name="OPERATION-FORCE" value="260g" x="-15" y="0" size="1.778" layer="27" display="off"/>
-<attribute name="PART-NUMBER" value="430162073826" x="-15" y="0" size="1.778" layer="27" display="off"/>
-<attribute name="QTY" value=" 250 " x="-15" y="0" size="1.778" layer="27" display="off"/>
-<attribute name="VALUE" value="430162073826" x="-18.494" y="-7.8258" size="1.27" layer="27"/>
-</element>
-<element name="S3" library="Wurth_Switch_WS-TASV" library_urn="urn:adsk.eagle:library:18304196" package="430162073826" package3d_urn="urn:adsk.eagle:package:18304357/2" value="430162073826" x="15" y="0" smashed="yes">
-<attribute name="DATASHEET-URL" value="https://www.we-online.com/redexpert/spec/430162073826?ae" x="15" y="0" size="1.778" layer="27" display="off"/>
-<attribute name="HEIGHT" value="7.3mm" x="15" y="0" size="1.778" layer="27" display="off"/>
+<attribute name="PART-NUMBER" value="430162043826" x="-15" y="0" size="1.778" layer="27" display="off"/>
+<attribute name="QTY" value=" 400 " x="-15" y="0" size="1.778" layer="27" display="off"/>
+<attribute name="VALUE" value="430162043826" x="-18.494" y="-7.8258" size="1.27" layer="27"/>
+</element>
+<element name="S3" library="Wurth_Switch_WS-TASV" library_urn="urn:adsk.eagle:library:18304196" package="430162043826" package3d_urn="urn:adsk.eagle:package:18304303/2" value="430162043826" x="15" y="0" smashed="yes">
+<attribute name="DATASHEET-URL" value="https://www.we-online.com/redexpert/spec/430162043826?ae" x="15" y="0" size="1.778" layer="27" display="off"/>
+<attribute name="HEIGHT" value="4.3mm" x="15" y="0" size="1.778" layer="27" display="off"/>
 <attribute name="NAME" x="14.966" y="6.9177" size="1.27" layer="25" align="bottom-center"/>
 <attribute name="OPERATION-FORCE" value="260g" x="15" y="0" size="1.778" layer="27" display="off"/>
-<attribute name="PART-NUMBER" value="430162073826" x="15" y="0" size="1.778" layer="27" display="off"/>
-<attribute name="QTY" value=" 250 " x="15" y="0" size="1.778" layer="27" display="off"/>
-<attribute name="VALUE" value="430162073826" x="11.506" y="-7.8258" size="1.27" layer="27"/>
-</element>
-<element name="S4" library="Wurth_Switch_WS-TASV" library_urn="urn:adsk.eagle:library:18304196" package="430162073826" package3d_urn="urn:adsk.eagle:package:18304357/2" value="430162073826" x="45" y="0" smashed="yes">
-<attribute name="DATASHEET-URL" value="https://www.we-online.com/redexpert/spec/430162073826?ae" x="45" y="0" size="1.778" layer="27" display="off"/>
-<attribute name="HEIGHT" value="7.3mm" x="45" y="0" size="1.778" layer="27" display="off"/>
+<attribute name="PART-NUMBER" value="430162043826" x="15" y="0" size="1.778" layer="27" display="off"/>
+<attribute name="QTY" value=" 400 " x="15" y="0" size="1.778" layer="27" display="off"/>
+<attribute name="VALUE" value="430162043826" x="11.506" y="-7.8258" size="1.27" layer="27"/>
+</element>
+<element name="S4" library="Wurth_Switch_WS-TASV" library_urn="urn:adsk.eagle:library:18304196" package="430162043826" package3d_urn="urn:adsk.eagle:package:18304303/2" value="430162043826" x="45" y="0" smashed="yes">
+<attribute name="DATASHEET-URL" value="https://www.we-online.com/redexpert/spec/430162043826?ae" x="45" y="0" size="1.778" layer="27" display="off"/>
+<attribute name="HEIGHT" value="4.3mm" x="45" y="0" size="1.778" layer="27" display="off"/>
 <attribute name="NAME" x="44.966" y="6.9177" size="1.27" layer="25" align="bottom-center"/>
 <attribute name="OPERATION-FORCE" value="260g" x="45" y="0" size="1.778" layer="27" display="off"/>
-<attribute name="PART-NUMBER" value="430162073826" x="45" y="0" size="1.778" layer="27" display="off"/>
-<attribute name="QTY" value=" 250 " x="45" y="0" size="1.778" layer="27" display="off"/>
-<attribute name="VALUE" value="430162073826" x="41.506" y="-7.8258" size="1.27" layer="27"/>
+<attribute name="PART-NUMBER" value="430162043826" x="45" y="0" size="1.778" layer="27" display="off"/>
+<attribute name="QTY" value=" 400 " x="45" y="0" size="1.778" layer="27" display="off"/>
+<attribute name="VALUE" value="430162043826" x="41.506" y="-7.8258" size="1.27" layer="27"/>
 </element>
 <element name="J2" library="Wurth_Connectors_WR-TBL Rising Cage Clamp" library_urn="urn:adsk.eagle:library:16280519" package="691709710305" package3d_urn="urn:adsk.eagle:package:16248446/4" value="691709710305" x="0" y="17.5" smashed="yes" rot="MR180">
