File: Hutschienenmoped-XL/Hauptplatine/Hauptplatine.brd (EAGLE design)
At the start: 96.3 x 101.8 mm, 138 parts, among them J1 638207222005, J13 638207222005, J15 638207222008, J2 645004114822, J4 61300421121, J7 638207222005, J8 638207222007, U4 TLE9250VSJ

Commit message: Updates resistor values and library URNs
Changes resistor values from 13k to 22k.

Updates library URNs in the eagle project file and board file.

Sets linktopcb3d to false in the board file.
Parts:
- R23, R26, R31, R32, R41, R44, R53, R56: value 13K -> 22K
Changed lines of the file:
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@@
 </layers>
 <board>
-<fusionsync huburn="a.YnVzaW5lc3M6bXNtdWM" projecturn="a.YnVzaW5lc3M6bXNtdWMjMjAyMjAzMTc1MDgxMzE4ODE" f3durn="urn:adsk.wipprod:dm.lineage:AZr2ohsdTDeaNf8dmFIMlA" pcbguid="" lastpulledtime="" lastsyncedchangeguid="" latestrevisionid="25d4beac-188d-4e0d-9dc1-4fed8a35951d" lastsyncedrevisionid="25d4beac-188d-4e0d-9dc1-4fed8a35951d" lastboardhashguid="84b5fabf-717a-1f2a-69b5-34e3e12fd72e" lastpushedtime="2024-07-16T14:49:39Z" linktopcb3d="true"/>
+<fusionsync huburn="a.YnVzaW5lc3M6bXNtdWM" projecturn="a.YnVzaW5lc3M6bXNtdWMjMjAyMjAzMTc1MDgxMzE4ODE" f3durn="urn:adsk.wipprod:dm.lineage:AZr2ohsdTDeaNf8dmFIMlA" pcbguid="" lastpulledtime="" lastsyncedchangeguid="" latestrevisionid="25d4beac-188d-4e0d-9dc1-4fed8a35951d" lastsyncedrevisionid="25d4beac-188d-4e0d-9dc1-4fed8a35951d" lastboardhashguid="84b5fabf-717a-1f2a-69b5-34e3e12fd72e" lastpushedtime="2024-07-16T14:49:39Z" linktopcb3d="false"/>
 <plain>
 <wire x1="52.04" y1="41.46" x2="50.54" y2="41.46" width="0.1524" layer="22"/>
@@
 <attribute name="WIDTH" value="1.6mm" x="46.99" y="65.405" size="1.778" layer="27" rot="R270" display="off"/>
 </element>
-<element name="R32" library="resistor" library_urn="urn:adsk.eagle:library:348" package="R1206" package3d_urn="urn:adsk.eagle:package:23540/2" value="13K" x="46.99" y="74.295" smashed="yes" rot="R270">
+<element name="R32" library="resistor" library_urn="urn:adsk.eagle:library:348" package="R1206" package3d_urn="urn:adsk.eagle:package:23540/2" value="22K" x="46.99" y="74.295" smashed="yes" rot="R270">
 <attribute name="NAME" x="47.54" y="74.345" size="0.3048" layer="25" rot="R270" align="bottom-center"/>
 </element>
@@
 <attribute name="WIDTH" value="1.6mm" x="49.53" y="65.405" size="1.778" layer="27" rot="R270" display="off"/>
 </element>
-<element name="R31" library="resistor" library_urn="urn:adsk.eagle:library:348" package="R1206" package3d_urn="urn:adsk.eagle:package:23540/2" value="13K" x="49.53" y="74.295" smashed="yes" rot="R270">
+<element name="R31" library="resistor" library_urn="urn:adsk.eagle:library:348" package="R1206" package3d_urn="urn:adsk.eagle:package:23540/2" value="22K" x="49.53" y="74.295" smashed="yes" rot="R270">
 <attribute name="NAME" x="50.08" y="74.345" size="0.3048" layer="25" rot="R270" align="bottom-center"/>
 </element>
@@
 <attribute name="WIDTH" value="1.6mm" x="16.51" y="65.405" size="1.778" layer="27" rot="R270" display="off"/>
 </element>
-<element name="R23" library="resistor" library_urn="urn:adsk.eagle:library:348" package="R1206" package3d_urn="urn:adsk.eagle:package:23540/2" value="13K" x="16.51" y="74.295" smashed="yes" rot="R270">
+<element name="R23" library="resistor" library_urn="urn:adsk.eagle:library:348" package="R1206" package3d_urn="urn:adsk.eagle:package:23540/2" value="22K" x="16.51" y="74.295" smashed="yes" rot="R270">
 <attribute name="NAME" x="17.06" y="74.345" size="0.3048" layer="25" rot="R270" align="bottom-center"/>
 </element>
@@
 <attribute name="WIDTH" value="1.6mm" x="19.05" y="65.405" size="1.778" layer="27" rot="R270" display="off"/>
 </element>
-<element name="R26" library="resistor" library_urn="urn:adsk.eagle:library:348" package="R1206" package3d_urn="urn:adsk.eagle:package:23540/2" value="13K" x="19.05" y="74.295" smashed="yes" rot="R270">
+<element name="R26" library="resistor" library_urn="urn:adsk.eagle:library:348" package="R1206" package3d_urn="urn:adsk.eagle:package:23540/2" value="22K" x="19.05" y="74.295" smashed="yes" rot="R270">
 <attribute name="NAME" x="19.6" y="74.345" size="0.3048" layer="25" rot="R270" align="bottom-center"/>
 </element>
@@
 <attribute name="WIDTH" value="1.6mm" x="26.67" y="65.405" size="1.778" layer="27" rot="R270" display="off"/>
 </element>
-<element name="R41" library="resistor" library_urn="urn:adsk.eagle:library:348" package="R1206" package3d_urn="urn:adsk.eagle:package:23540/2" value="13K" x="26.67" y="74.295" smashed="yes" rot="R270">
+<element name="R41" library="resistor" library_urn="urn:adsk.eagle:library:348" package="R1206" package3d_urn="urn:adsk.eagle:package:23540/2" value="22K" x="26.67" y="74.295" smashed="yes" rot="R270">
 <attribute name="NAME" x="27.22" y="74.345" size="0.3048" layer="25" rot="R270" align="bottom-center"/>
 </element>
@@
 <attribute name="WIDTH" value="1.6mm" x="31.75" y="65.405" size="1.778" layer="27" rot="R270" display="off"/>
 </element>
-<element name="R44" library="resistor" library_urn="urn:adsk.eagle:library:348" package="R1206" package3d_urn="urn:adsk.eagle:package:23540/2" value="13K" x="31.75" y="74.295" smashed="yes" rot="R270">
+<element name="R44" library="resistor" library_urn="urn:adsk.eagle:library:348" package="R1206" package3d_urn="urn:adsk.eagle:package:23540/2" value="22K" x="31.75" y="74.295" smashed="yes" rot="R270">
 <attribute name="NAME" x="32.3" y="74.345" size="0.3048" layer="25" rot="R270" align="bottom-center"/>
 </element>
@@
 <attribute name="WIDTH" value="1.6mm" x="36.83" y="65.405" size="1.778" layer="27" rot="R270" display="off"/>
 </element>
-<element name="R53" library="resistor" library_urn="urn:adsk.eagle:library:348" package="R1206" package3d_urn="urn:adsk.eagle:package:23540/2" value="13K" x="36.83" y="74.295" smashed="yes" rot="R270">
+<element name="R53" library="resistor" library_urn="urn:adsk.eagle:library:348" package="R1206" package3d_urn="urn:adsk.eagle:package:23540/2" value="22K" x="36.83" y="74.295" smashed="yes" rot="R270">
 <attribute name="NAME" x="37.38" y="74.345" size="0.3048" layer="25" rot="R270" align="bottom-center"/>
 </element>
@@
 <attribute name="WIDTH" value="1.6mm" x="39.37" y="65.405" size="1.778" layer="27" rot="R270" display="off"/>
 </element>
-<element name="R56" library="resistor" library_urn="urn:adsk.eagle:library:348" package="R1206" package3d_urn="urn:adsk.eagle:package:23540/2" value="13K" x="39.37" y="74.295" smashed="yes" rot="R270">
+<element name="R56" library="resistor" library_urn="urn:adsk.eagle:library:348" package="R1206" package3d_urn="urn:adsk.eagle:package:23540/2" value="22K" x="39.37" y="74.295" smashed="yes" rot="R270">
 <attribute name="NAME" x="39.92" y="74.345" size="0.3048" layer="25" rot="R270" align="bottom-center"/>
 </element>
